Commit message: L10 Right URDF Updated

File: l10/right/linkerhand_l10_right.urdf (robot description, URDF)
Before this commit: robot linker_hand_l10_right, 26 links, 25 joints
Links:
- removed link base_link
- removed link index_link0
- removed link index_link1
- removed link index_link2
- removed link index_link3
- removed link index_link4
- removed link little_link0
- removed link little_link1
- removed link little_link2
- removed link little_link3
- removed link little_link4
- removed link middle_link0
- removed link middle_link1
- removed link middle_link2
- removed link middle_link3
- removed link ring_link0
- removed link ring_link1
- removed link ring_link2
- removed link ring_link3
- removed link ring_link4
- removed link thumb_link0
- removed link thumb_link1
- removed link thumb_link2
- removed link thumb_link3
- removed link thumb_link4
- removed link thumb_link5
- added link hand_base_link, mass 0.34354881926881575; collision mesh filename=meshes/hand_base_link.STL; visual mesh filename=meshes/hand_base_link.STL
- added link index_distal, mass 0.014858278875807667; collision mesh filename=meshes/index_distal.STL; visual mesh filename=meshes/index_distal.STL
- added link index_metacarpals, mass 0.016614213530707737; collision mesh filename=meshes/index_metacarpals.STL; visual mesh filename=meshes/index_metacarpals.STL
- added link index_middle, mass 0.012511711108351411; collision mesh filename=meshes/index_middle.STL; visual mesh filename=meshes/index_middle.STL
- added link index_proximal, mass 0.01170870731662533; collision mesh filename=meshes/index_proximal.STL; visual mesh filename=meshes/index_proximal.STL
- added link middle_distal, mass 0.014858277037854526; collision mesh filename=meshes/middle_distal.STL; visual mesh filename=meshes/middle_distal.STL
- added link middle_middle, mass 0.012511710480750374; collision mesh filename=meshes/middle_middle.STL; visual mesh filename=meshes/middle_middle.STL
- added link middle_proximal, mass 0.011708689871923124; collision mesh filename=meshes/middle_proximal.STL; visual mesh filename=meshes/middle_proximal.STL
- added link pinky_distal, mass 0.014858275630682649; collision mesh filename=meshes/pinky_distal.STL; visual mesh filename=meshes/pinky_distal.STL
- added link pinky_metacarpals, mass 0.01661421467628334; collision mesh filename=meshes/pinky_metacarpals.STL; visual mesh filename=meshes/pinky_metacarpals.STL
- added link pinky_middle, mass 0.01251170901822359; collision mesh filename=meshes/pinky_middle.STL; visual mesh filename=meshes/pinky_middle.STL
- added link pinky_proximal, mass 0.011736005978942131; collision mesh filename=meshes/pinky_proximal.STL; visual mesh filename=meshes/pinky_proximal.STL
- added link ring_distal, mass 0.014858274891747264; collision mesh filename=meshes/ring_distal.STL; visual mesh filename=meshes/ring_distal.STL
- added link ring_metacarpals, mass 0.016614214319408793; collision mesh filename=meshes/ring_metacarpals.STL; visual mesh filename=meshes/ring_metacarpals.STL
- added link ring_middle, mass 0.012511709056521332; collision mesh filename=meshes/ring_middle.STL; visual mesh filename=meshes/ring_middle.STL
- added link ring_proximal, mass 0.011708644033664218; collision mesh filename=meshes/ring_proximal.STL; visual mesh filename=meshes/ring_proximal.STL
- added link thumb_distal, mass 0.023012842812374323; collision mesh filename=meshes/thumb_distal.STL; visual mesh filename=meshes/thumb_distal.STL
- added link thumb_metacarpals, mass 0.0681681057244462; collision mesh filename=meshes/thumb_metacarpals.STL; visual mesh filename=meshes/thumb_metacarpals.STL
- added link thumb_metacarpals_base1, mass 0.04425566779982592; collision mesh filename=meshes/thumb_metacarpals_base1.STL; visual mesh filename=meshes/thumb_metacarpals_base1.STL
- added link thumb_metacarpals_base2, mass 0.06546850411934668; collision mesh filename=meshes/thumb_metacarpals_base2.STL; visual mesh filename=meshes/thumb_metacarpals_base2.STL
- added link thumb_proximal, mass 0.020057039570174552; collision mesh filename=meshes/thumb_proximal.STL; visual mesh filename=meshes/thumb_proximal.STL
Joints:
- removed joint index_joint0
- removed joint index_joint1
- removed joint index_joint2
- removed joint index_joint3
- removed joint index_joint4
- removed joint little_joint0
- removed joint little_joint1
- removed joint little_joint2
- removed joint little_joint3
- removed joint little_joint4
- removed joint middle_joint0
- removed joint middle_joint1
- removed joint middle_joint2
- removed joint middle_joint3
- removed joint ring_joint0
- removed joint ring_joint1
- removed joint ring_joint2
- removed joint ring_joint3
- removed joint ring_joint4
- removed joint thumb_joint0
- removed joint thumb_joint1
- removed joint thumb_joint2
- removed joint thumb_joint3
- removed joint thumb_joint4
- removed joint thumb_joint5
- added joint index_dip: type revolute, parent index_middle, child index_distal, origin xyz=-0.0050438 0 0.025752 rpy=0 0 0, axis 0 1 0, limit lower=0 upper=1 effort=100 velocity=1, mimic joint=index_pip multiplier=0.635 offset=0
- added joint index_mcp_pitch: type revolute, parent index_metacarpals, child index_proximal, origin xyz=0.0010297 0 0.017575 rpy=0 0 0, axis 0 1 0, limit lower=0 upper=1.325 effort=100 velocity=1
- added joint index_mcp_roll: type revolute, parent hand_base_link, child index_metacarpals, origin xyz=-0.0021525 0.02293 0.12973 rpy=-0.0017399 0 0, axis 1 0 0, limit lower=-0.36 upper=0.36 effort=100 velocity=1
- added joint index_pip: type revolute, parent index_proximal, child index_middle, origin xyz=-0.0033727 0 0.03351 rpy=0 0 0, axis 0 1 0, limit lower=0 upper=1.57 effort=100 velocity=1, mimic joint=index_mcp_pitch multiplier=1.18 offset=0
- added joint middle_dip: type revolute, parent middle_middle, child middle_distal, origin xyz=-0.0050438 0 0.025752 rpy=0 0 0, axis 0 1 0, limit lower=0 upper=1 effort=100 velocity=1, mimic joint=middle_pip multiplier=0.635 offset=0
- added joint middle_mcp_pitch: type revolute, parent hand_base_link, child middle_proximal, origin xyz=-0.0031229 0.0039297 0.1523 rpy=0 0 0, axis 0 1 0, limit lower=0 upper=1.325 effort=100 velocity=1
- added joint middle_pip: type revolute, parent middle_proximal, child middle_middle, origin xyz=-0.0033727 0 0.03351 rpy=0 0 0, axis 0 1 0, limit lower=0 upper=1.57 effort=100 velocity=1, mimic joint=middle_mcp_pitch multiplier=1.18 offset=0
- added joint pinky_dip: type revolute, parent pinky_middle, child pinky_distal, origin xyz=-0.0050438 0 0.025752 rpy=0 0 0, axis 0 1 0, limit lower=0 upper=1 effort=100 velocity=1, mimic joint=pinky_pip multiplier=0.635 offset=0
- added joint pinky_mcp_pitch: type revolute, parent pinky_metacarpals, child pinky_proximal, origin xyz=0.0010315 0 0.017575 rpy=0 0 0, axis 0 1 0, limit lower=0 upper=1.325 effort=100 velocity=1
- added joint pinky_mcp_roll: type revolute, parent hand_base_link, child pinky_metacarpals, origin xyz=-0.00015438 -0.03407 0.12473 rpy=0.0073744 0 0, axis 1 0 0, limit lower=-0.36 upper=0.36 effort=100 velocity=1
- added joint pinky_pip: type revolute, parent pinky_proximal, child pinky_middle, origin xyz=-0.0033727 0 0.03351 rpy=0 0 0, axis 0 1 0, limit lower=0 upper=1.57 effort=100 velocity=1, mimic joint=pinky_mcp_pitch multiplier=1.18 offset=0
- added joint ring_dip: type revolute, parent ring_middle, child ring_distal, origin xyz=-0.0050438 0 0.025752 rpy=0 0 0, axis 0 1 0, limit lower=0 upper=1 effort=100 velocity=1, mimic joint=ring_pip multiplier=0.635 offset=0
- added joint ring_mcp_pitch: type revolute, parent ring_metacarpals, child ring_proximal, origin xyz=0.0010315 0 0.017575 rpy=0 0 0, axis 0 1 0, limit lower=0 upper=1.325 effort=100 velocity=1
- added joint ring_mcp_roll: type revolute, parent hand_base_link, child ring_metacarpals, origin xyz=-0.0021544 -0.01507 0.12973 rpy=0.004655 0 0, axis 1 0 0, limit lower=-0.36 upper=0.36 effort=100 velocity=1
- added joint ring_pip: type revolute, parent ring_proximal, child ring_middle, origin xyz=-0.0033727 0 0.03351 rpy=0 0 0, axis 0 1 0, limit lower=0 upper=1.57 effort=100 velocity=1, mimic joint=ring_mcp_pitch multiplier=1.18 offset=0
- added joint thumb_cmc_pitch: type revolute, parent thumb_metacarpals_base2, child thumb_metacarpals, origin xyz=5.9553E-05 0.0034929 0.028731 rpy=0 0.46329 -1.5708, axis 0 1 0, limit lower=0 upper=0.5286 effort=100 velocity=1
- added joint thumb_cmc_roll: type revolute, parent hand_base_link, child thumb_metacarpals_base1, origin xyz=-0.016657 0.018426 0.057469 rpy=0 0 0, axis 1 0 0, limit lower=-0.785 upper=0.785 effort=100 velocity=1
- added joint thumb_cmc_yaw: type revolute, parent thumb_metacarpals_base1, child thumb_metacarpals_base2, origin xyz=0.029035 -1.086E-05 0.0020117 rpy=-1.5708 0 -0.56048, axis 0 1 0, limit lower=0 upper=1.57 effort=100 velocity=1
- added joint thumb_ip: type revolute, parent thumb_proximal, child thumb_distal, origin xyz=-0.0040391 0 0.036444 rpy=0 0 0, axis 0 1 0, limit lower=0 upper=1.256 effort=100 velocity=1, mimic joint=thumb_mcp multiplier=1.0625 offset=0
- added joint thumb_mcp: type revolute, parent thumb_metacarpals, child thumb_proximal, origin xyz=0.0049422 0 0.050268 rpy=0 0 0, axis 0 1 0, limit lower=0 upper=1.0467 effort=100 velocity=1, mimic joint=thumb_cmc_pitch multiplier=2.24 offset=0

Commit message: L10 double updated

File: l10/right/linkerhand_l10_right.urdf (robot description, URDF)
Before this commit: robot linkerhand_l10_right.urdf, 21 links, 20 joints
Joints:
- joint index_dip: limit lower=0 upper=1 effort=100 velocity=1 -> lower=0 upper=1 effort=12 velocity=2.6
- joint index_mcp_pitch: limit lower=0 upper=1.325 effort=100 velocity=1 -> lower=0 upper=1.325 effort=12 velocity=2.6
- joint index_mcp_roll: limit lower=-0.36 upper=0.36 effort=100 velocity=1 -> lower=-0.36 upper=0.36 effort=12 velocity=2.6
- joint index_pip: limit lower=0 upper=1.57 effort=100 velocity=1 -> lower=0 upper=1.57 effort=12 velocity=2.6
- joint middle_dip: limit lower=0 upper=1 effort=100 velocity=1 -> lower=0 upper=1 effort=12 velocity=2.6
- joint middle_mcp_pitch: limit lower=0 upper=1.325 effort=100 velocity=1 -> lower=0 upper=1.325 effort=12 velocity=2.6
- joint middle_pip: limit lower=0 upper=1.57 effort=100 velocity=1 -> lower=0 upper=1.57 effort=12 velocity=2.6
- joint pinky_dip: limit lower=0 upper=1 effort=100 velocity=1 -> lower=0 upper=1 effort=12 velocity=2.6
- joint pinky_mcp_pitch: limit lower=0 upper=1.325 effort=100 velocity=1 -> lower=0 upper=1.325 effort=12 velocity=2.6
- joint pinky_mcp_roll: limit lower=-0.36 upper=0.36 effort=100 velocity=1 -> lower=-0.36 upper=0.36 effort=12 velocity=2.6
- joint pinky_pip: limit lower=0 upper=1.57 effort=100 velocity=1 -> lower=0 upper=1.57 effort=12 velocity=2.6
- joint ring_dip: limit lower=0 upper=1 effort=100 velocity=1 -> lower=0 upper=1 effort=12 velocity=2.6
- joint ring_mcp_pitch: limit lower=0 upper=1.325 effort=100 velocity=1 -> lower=0 upper=1.325 effort=12 velocity=2.6
- joint ring_mcp_roll: limit lower=-0.36 upper=0.36 effort=100 velocity=1 -> lower=-0.36 upper=0.36 effort=12 velocity=2.6
- joint ring_pip: limit lower=0 upper=1.57 effort=100 velocity=1 -> lower=0 upper=1.57 effort=12 velocity=2.6
- joint thumb_cmc_pitch: limit lower=0 upper=0.5286 effort=100 velocity=1 -> lower=0 upper=0.5286 effort=12 velocity=2.6
- joint thumb_cmc_roll: limit lower=-0.785 upper=0.785 effort=100 velocity=1 -> lower=-0.785 upper=0.785 effort=12 velocity=2.6
- joint thumb_cmc_yaw: limit lower=0 upper=1.57 effort=100 velocity=1 -> lower=0 upper=1.57 effort=12 velocity=2.6
- joint thumb_ip: limit lower=0 upper=1.256 effort=100 velocity=1 -> lower=0 upper=1.256 effort=12 velocity=2.6
- joint thumb_mcp: limit lower=0 upper=1.0467 effort=100 velocity=1 -> lower=0 upper=1.0467 effort=12 velocity=2.6
