Commit message: update o7v3 urdf

File: o7v3/left/linkerhand_o7v3_left.urdf (robot description, URDF)
Before this commit: robot linkerhand_O7_left.urdf, 18 links, 17 joints
Joints:
- joint index_dip: limit lower=0 upper=0.628 effort=100 velocity=1 -> lower=0 upper=0.6053 effort=100 velocity=1; mimic joint=index_mcp_pitch multiplier=0.4615 offset=0 -> joint=index_mcp_pitch multiplier=0.46 offset=0
- joint index_mcp_pitch: limit lower=0 upper=1.3607 effort=100 velocity=1 -> lower=0 upper=1.3275 effort=100 velocity=1
- joint index_pip: limit lower=0 upper=1.8317 effort=100 velocity=1 -> lower=0 upper=1.7915 effort=100 velocity=1; mimic joint=index_mcp_pitch multiplier=1.3462 offset=0 -> joint=index_mcp_pitch multiplier=1.35 offset=0
- joint middle_distal: limit lower=0 upper=0.628 effort=100 velocity=1 -> lower=0 upper=0.6053 effort=100 velocity=1; mimic joint=middle_mcp_pitch multiplier=0.4615 offset=0 -> joint=middle_mcp_pitch multiplier=0.46 offset=0
- joint middle_mcp_pitch: limit lower=0 upper=1.3607 effort=100 velocity=1 -> lower=0 upper=1.3275 effort=100 velocity=1
- joint middle_pip: limit lower=0 upper=1.8317 effort=100 velocity=1 -> lower=0 upper=1.7915 effort=100 velocity=1; mimic joint=middle_mcp_pitch multiplier=1.3462 offset=0 -> joint=middle_mcp_pitch multiplier=1.35 offset=0
- joint pinky_dip: limit lower=0 upper=0.628 effort=100 velocity=1 -> lower=0 upper=0.6053 effort=100 velocity=1; mimic joint=pinky_mcp_pitch multiplier=0.4615 offset=0 -> joint=pinky_mcp_pitch multiplier=0.46 offset=0
- joint pinky_mcp_pitch: limit lower=0 upper=1.3607 effort=100 velocity=1 -> lower=0 upper=1.3275 effort=100 velocity=1
- joint pinky_pip: limit lower=0 upper=1.8317 effort=100 velocity=1 -> lower=0 upper=1.7915 effort=100 velocity=1; mimic joint=pinky_mcp_pitch multiplier=1.3462 offset=0 -> joint=pinky_mcp_pitch multiplier=1.35 offset=0
- joint ring_dip: limit lower=0 upper=0.628 effort=100 velocity=1 -> lower=0 upper=0.6053 effort=100 velocity=1; mimic joint=ring_mcp_pitch multiplier=0.4615 offset=0 -> joint=ring_mcp_pitch multiplier=0.46 offset=0
- joint ring_mcp_pitch: limit lower=0 upper=1.3607 effort=100 velocity=1 -> lower=0 upper=1.3275 effort=100 velocity=1
- joint ring_pip: limit lower=0 upper=1.8317 effort=100 velocity=1 -> lower=0 upper=1.7915 effort=100 velocity=1; mimic joint=ring_mcp_pitch multiplier=1.3462 offset=0 -> joint=ring_mcp_pitch multiplier=1.35 offset=0
- joint thumb_cmc_pitch: limit lower=0 upper=0.5146 effort=100 velocity=1 -> lower=0 upper=0.4867 effort=100 velocity=1
- joint thumb_cmc_roll: limit lower=0 upper=1.1339 effort=100 velocity=1 -> lower=0 upper=1.0467 effort=100 velocity=1
- joint thumb_cmc_yaw: limit lower=0 upper=1.9189 effort=100 velocity=1 -> lower=0 upper=1.2037 effort=100 velocity=1
- joint thumb_ip: limit lower=0 upper=0.7763 effort=100 velocity=1 -> lower=0 upper=0.6611 effort=100 velocity=1; mimic joint=thumb_cmc_pitch multiplier=1.5085 offset=0 -> joint=thumb_cmc_pitch multiplier=1.36 offset=0
- joint thumb_mcp: limit lower=0 upper=0.7152 effort=100 velocity=1 -> lower=0 upper=0.6699 effort=100 velocity=1; mimic joint=thumb_cmc_pitch multiplier=1.3898 offset=0 -> joint=thumb_cmc_pitch multiplier=1.38 offset=0

File: o7v3/right/linkerhand_o7v3_right.urdf (robot description, URDF)
Before this commit: robot linkerhand_O7_right.urdf, 18 links, 17 joints
Joints:
- joint index_dip: limit lower=0 upper=0.638 effort=100 velocity=1 -> lower=0 upper=0.6053 effort=100 velocity=1; mimic joint=index_mcp_pitch multiplier=0.4615 offset=0 -> joint=index_mcp_pitch multiplier=0.46 offset=0
- joint index_mcp_pitch: limit lower=0 upper=1.3607 effort=100 velocity=1 -> lower=0 upper=1.3275 effort=100 velocity=1
- joint index_pip: limit lower=0 upper=1.8317 effort=100 velocity=1 -> lower=0 upper=1.7915 effort=100 velocity=1; mimic joint=index_mcp_pitch multiplier=1.3462 offset=0 -> joint=index_mcp_pitch multiplier=1.35 offset=0
- joint middle_dip: limit lower=0 upper=0.628 effort=100 velocity=1 -> lower=0 upper=0.6053 effort=100 velocity=1; mimic joint=middle_mcp_pitch multiplier=0.4615 offset=0 -> joint=middle_mcp_pitch multiplier=0.46 offset=0
- joint middle_mcp_pitch: limit lower=0 upper=1.3607 effort=100 velocity=1 -> lower=0 upper=1.3275 effort=100 velocity=1
- joint middle_pip: limit lower=0 upper=1.8317 effort=100 velocity=1 -> lower=0 upper=1.7915 effort=100 velocity=1; mimic joint=middle_mcp_pitch multiplier=1.3462 offset=0 -> joint=middle_mcp_pitch multiplier=1.35 offset=0
- joint pinky_dip: limit lower=0 upper=0.628 effort=100 velocity=1 -> lower=0 upper=0.6053 effort=100 velocity=1; mimic joint=pinky_mcp_pitch multiplier=0.4615 offset=0 -> joint=pinky_mcp_pitch multiplier=0.46 offset=0
- joint pinky_mcp_pitch: limit lower=0 upper=1.3607 effort=100 velocity=1 -> lower=0 upper=1.3275 effort=100 velocity=1
- joint pinky_pip: limit lower=0 upper=1.8317 effort=100 velocity=1 -> lower=0 upper=1.7915 effort=100 velocity=1; mimic joint=pinky_mcp_pitch multiplier=1.3462 offset=0 -> joint=pinky_mcp_pitch multiplier=1.35 offset=0
- joint ring_dip: limit lower=0 upper=0.628 effort=100 velocity=1 -> lower=0 upper=0.6053 effort=100 velocity=1; mimic joint=ring_mcp_pitch multiplier=0.4615 offset=0 -> joint=ring_mcp_pitch multiplier=0.46 offset=0
- joint ring_mcp_pitch: limit lower=0 upper=1.3607 effort=100 velocity=1 -> lower=0 upper=1.3275 effort=100 velocity=1
- joint ring_pip: limit lower=0 upper=1.8317 effort=100 velocity=1 -> lower=0 upper=1.7915 effort=100 velocity=1; mimic joint=ring_mcp_pitch multiplier=1.3462 offset=0 -> joint=ring_mcp_pitch multiplier=1.35 offset=0
- joint thumb_cmc_pitch: limit lower=0 upper=0.5146 effort=100 velocity=1 -> lower=0 upper=0.4867 effort=100 velocity=1
- joint thumb_cmc_roll: limit lower=0 upper=1.1339 effort=100 velocity=1 -> lower=0 upper=1.0467 effort=100 velocity=1
- joint thumb_cmc_yaw: limit lower=0 upper=1.9189 effort=100 velocity=1 -> lower=0 upper=1.2037 effort=100 velocity=1
- joint thumb_ip: limit lower=0 upper=0.7763 effort=100 velocity=1 -> lower=0 upper=0.6611 effort=100 velocity=1; mimic joint=thumb_cmc_pitch multiplier=1.5085 offset=0 -> joint=thumb_cmc_pitch multiplier=1.36 offset=0
- joint thumb_mcp: limit lower=0 upper=0.7152 effort=100 velocity=1 -> lower=0 upper=0.6699 effort=100 velocity=1; mimic joint=thumb_cmc_pitch multiplier=1.3898 offset=0 -> joint=thumb_cmc_pitch multiplier=1.38 offset=0
