Commit message: update l20 urdf

File: l20/left/linkerhand_l20_left.urdf (robot description, URDF)
Before this commit: robot linker_hand_l20_left, 27 links, 26 joints
Links:
- removed link base_link
- removed link index_link0
- removed link index_link1
- removed link index_link2
- removed link index_link3
- removed link index_link4
- removed link little_link0
- removed link little_link1
- removed link little_link2
- removed link little_link3
- removed link little_link4
- removed link middle_link0
- removed link middle_link1
- removed link middle_link2
- removed link middle_link3
- removed link middle_link4
- removed link ring_link0
- removed link ring_link1
- removed link ring_link2
- removed link ring_link3
- removed link ring_link4
- removed link thumb_link0
- removed link thumb_link1
- removed link thumb_link2
- removed link thumb_link3
- removed link thumb_link4
- removed link thumb_link5
- added link hand_base_link, mass 0.101492069055989; collision mesh filename=meshes/hand_base_link.STL; visual mesh filename=meshes/hand_base_link.STL
- added link index_distal, mass 0.00386200107962104; collision mesh filename=meshes/index_distal.STL; visual mesh filename=meshes/index_distal.STL
- added link index_metacarpals, mass 0.000826416925828409; collision mesh filename=meshes/index_metacarpals.STL; visual mesh filename=meshes/index_metacarpals.STL
- added link index_middle, mass 0.0018096470933759; collision mesh filename=meshes/index_middle.STL; visual mesh filename=meshes/index_middle.STL
- added link index_proximal, mass 0.00454034378439372; collision mesh filename=meshes/index_proximal.STL; visual mesh filename=meshes/index_proximal.STL
- added link middle_distal, mass 0.00386200248743799; collision mesh filename=meshes/middle_distal.STL; visual mesh filename=meshes/middle_distal.STL
- added link middle_metacarpals, mass 0.000826416925828398; collision mesh filename=meshes/middle_metacarpals.STL; visual mesh filename=meshes/middle_metacarpals.STL
- added link middle_middle, mass 0.00180964709329765; collision mesh filename=meshes/middle_middle.STL; visual mesh filename=meshes/middle_middle.STL
- added link middle_proximal, mass 0.00454034378346624; collision mesh filename=meshes/middle_proximal.STL; visual mesh filename=meshes/middle_proximal.STL
- added link pinky_distal, mass 0.00386200247559812; collision mesh filename=meshes/pinky_distal.STL; visual mesh filename=meshes/pinky_distal.STL
- added link pinky_metacarpals, mass 0.000826416925828368; collision mesh filename=meshes/pinky_metacarpals.STL; visual mesh filename=meshes/pinky_metacarpals.STL
- added link pinky_middle, mass 0.00180964709325975; collision mesh filename=meshes/pinky_middle.STL; visual mesh filename=meshes/pinky_middle.STL
- added link pinky_proximal, mass 0.00454034378334877; collision mesh filename=meshes/pinky_proximal.STL; visual mesh filename=meshes/pinky_proximal.STL
- added link ring_distal, mass 0.00386200102769892; collision mesh filename=meshes/ring_distal.STL; visual mesh filename=meshes/ring_distal.STL
- added link ring_metacarpals, mass 0.000826416925828383; collision mesh filename=meshes/ring_metacarpals.STL; visual mesh filename=meshes/ring_metacarpals.STL
- added link ring_middle, mass 0.00180964709329766; collision mesh filename=meshes/ring_middle.STL; visual mesh filename=meshes/ring_middle.STL
- added link ring_proximal, mass 0.00454034378337052; collision mesh filename=meshes/ring_proximal.STL; visual mesh filename=meshes/ring_proximal.STL
- added link thumb_distal, mass 0.00432493724895246; collision mesh filename=meshes/thumb_distal.STL; visual mesh filename=meshes/thumb_distal.STL
- added link thumb_metacarpals, mass 0.0120240677638171; collision mesh filename=meshes/thumb_metacarpals.STL; visual mesh filename=meshes/thumb_metacarpals.STL
- added link thumb_metacarpals_base1, mass 0.00274839797669793; collision mesh filename=meshes/thumb_metacarpals_base1.STL; visual mesh filename=meshes/thumb_metacarpals_base1.STL
- added link thumb_metacarpals_base2, mass 0.00427940802750865; collision mesh filename=meshes/thumb_metacarpals_base2.STL; visual mesh filename=meshes/thumb_metacarpals_base2.STL
- added link thumb_proximal, mass 0.00531602156580031; collision mesh filename=meshes/thumb_proximal.STL; visual mesh filename=meshes/thumb_proximal.STL
Joints:
- removed joint index_joint0
- removed joint index_joint1
- removed joint index_joint2
- removed joint index_joint3
- removed joint index_joint4
- removed joint little_joint0
- removed joint little_joint1
- removed joint little_joint2
- removed joint little_joint3
- removed joint little_joint4
- removed joint middle_joint0
- removed joint middle_joint1
- removed joint middle_joint2
- removed joint middle_joint3
- removed joint middle_joint4
- removed joint ring_joint0
- removed joint ring_joint1
- removed joint ring_joint2
- removed joint ring_joint3
- removed joint ring_joint4
- removed joint thumb_joint0
- removed joint thumb_joint1
- removed joint thumb_joint2
- removed joint thumb_joint3
- removed joint thumb_joint4
- removed joint thumb_joint5
- added joint index_dip: type revolute, parent index_middle, child index_distal, origin xyz=0.00275581955818074 0 0.0317033719231916 rpy=0 0 0, axis 0 0.999999999999978 0, limit lower=0 upper=1.43 effort=100 velocity=1, mimic joint=index_pip multiplier=0.807909 offset=0
- added joint index_mcp_pitch: type revolute, parent index_metacarpals, child index_proximal, origin xyz=0.01087006638288 -1.2630433198893E-05 0 rpy=0 0 0, axis 0 0.999999999999978 0, limit lower=0 upper=1.33 effort=100 velocity=1
- added joint index_mcp_roll: type revolute, parent hand_base_link, child index_metacarpals, origin xyz=-0.0236662629253359 -0.0267021153669649 0.159311473821529 rpy=0 0 0, axis 0.999999999999989 0 0, limit lower=-0.18 upper=0.18 effort=100 velocity=1
- added joint index_pip: type revolute, parent index_proximal, child index_middle, origin xyz=-0.00419480624913221 0 0.0448194128870992 rpy=0 0 0, axis 0 0.999999999999978 0, limit lower=0 upper=1.77 effort=100 velocity=1
- added joint middle_dip: type revolute, parent middle_middle, child middle_distal, origin xyz=0.00275581955816206 0 0.0317033719231916 rpy=0 0 0, axis 0 0.999999999997063 0, limit lower=0 upper=1.43 effort=100 velocity=1, mimic joint=middle_pip multiplier=0.807909 offset=0
- added joint middle_mcp_pitch: type revolute, parent middle_metacarpals, child middle_proximal, origin xyz=0.0108700663541581 -1.26551278382542E-05 0 rpy=0 0 0, axis 0 0.999999999997063 0, limit lower=0 upper=1.33 effort=100 velocity=1
- added joint middle_mcp_roll: type revolute, parent hand_base_link, child middle_metacarpals, origin xyz=-0.028550041829013 -0.00510211872877702 0.163804366151529 rpy=0 0 0, axis 0.999999999997074 0 0, limit lower=-0.18 upper=0.18 effort=100 velocity=1
- added joint middle_pip: type revolute, parent middle_proximal, child middle_middle, origin xyz=-0.00419480624913501 0 0.0448194128870992 rpy=0 0 0, axis 0 0.999999999997063 0, limit lower=0 upper=1.77 effort=100 velocity=1
- added joint pinky_dip: type revolute, parent pinky_middle, child pinky_distal, origin xyz=0.00275581955821799 0 0.0317033719231203 rpy=0 0 0, axis 0 0.999999999997607 0, limit lower=0 upper=1.43 effort=100 velocity=1, mimic joint=pinky_pip multiplier=0.807909 offset=0
- added joint pinky_mcp_pitch: type revolute, parent pinky_metacarpals, child pinky_proximal, origin xyz=0.0108700663781205 -1.26345288001539E-05 0 rpy=0 0 0, axis 0 0.999999999997607 0, limit lower=0 upper=1.33 effort=100 velocity=1
- added joint pinky_mcp_roll: type revolute, parent hand_base_link, child pinky_metacarpals, origin xyz=-0.0226215026189916 0.0380979799565023 0.150312739475098 rpy=0 0 0, axis 0.999999999999863 0 0, limit lower=-0.18 upper=0.18 effort=100 velocity=1
- added joint pinky_pip: type revolute, parent pinky_proximal, child pinky_middle, origin xyz=-0.00419480624907856 0 0.0448194128869988 rpy=0 0 0, axis 0 0.999999999997607 0, limit lower=0 upper=1.77 effort=100 velocity=1
- added joint ring_dip: type revolute, parent ring_middle, child ring_distal, origin xyz=0.00275581955816206 0 0.0317033719231916 rpy=0 0 0, axis 0 0.999999999997063 0, limit lower=0 upper=1.43 effort=100 velocity=1, mimic joint=ring_pip multiplier=0.807909 offset=0
- added joint ring_mcp_pitch: type revolute, parent ring_metacarpals, child ring_proximal, origin xyz=0.0108700663541581 -1.26551278382542E-05 0 rpy=0 0 0, axis 0 0.999999999997063 0, limit lower=0 upper=1.33 effort=100 velocity=1
- added joint ring_mcp_roll: type revolute, parent hand_base_link, child ring_metacarpals, origin xyz=-0.026245256656013 0.016497885055223 0.159311479072529 rpy=0 0 0, axis 0.999999999997074 0 0, limit lower=-0.18 upper=0.18 effort=100 velocity=1
- added joint ring_pip: type revolute, parent ring_proximal, child ring_middle, origin xyz=-0.00419480624913501 0 0.0448194128870992 rpy=0 0 0, axis 0 0.999999999997063 0, limit lower=0 upper=1.77 effort=100 velocity=1
- added joint thumb_cmc_pitch: type revolute, parent thumb_metacarpals_base2, child thumb_metacarpals, origin xyz=0 -0.0307945049899851 0.00396440225285005 rpy=0 -0.767096499588843 1.57079617863246, axis 0 1 0, limit lower=0 upper=0.6 effort=100 velocity=1
- added joint thumb_cmc_roll: type revolute, parent hand_base_link, child thumb_metacarpals_base1, origin xyz=-0.000566250268316748 -0.00508587816314111 0.0573919459698274 rpy=0 0 0, axis -0.999999999999989 0 0, limit lower=-0.5 upper=0.8 effort=100 velocity=1
- added joint thumb_cmc_yaw: type revolute, parent thumb_metacarpals_base1, child thumb_metacarpals_base2, origin xyz=0.0245077602402008 -0.000833339999216351 0 rpy=0 0 0, axis 0 0 0.999999999999989, limit lower=0.15 upper=2.2 effort=100 velocity=1
- added joint thumb_ip: type revolute, parent thumb_proximal, child thumb_distal, origin xyz=-0.00294430789962509 0 0.0344361391557164 rpy=0 0 0, axis 0 1 0, limit lower=0 upper=1.2 effort=100 velocity=1, mimic joint=thumb_mcp multiplier=1 offset=0
- added joint thumb_mcp: type revolute, parent thumb_metacarpals, child thumb_proximal, origin xyz=0.00467511679938065 0.00010004081575718 0.0560361883792787 rpy=0 0 0, axis 0 1 0, limit lower=0 upper=1.2 effort=100 velocity=1

File: l20/right/linkerhand_l20_right.urdf (robot description, URDF)
Before this commit: robot linker_hand_l20_right, 27 links, 26 joints
Links:
- removed link index_link0
- removed link index_link1
- removed link index_link2
- removed link index_link3
- removed link index_link4
- removed link little_link0
- removed link little_link1
- removed link little_link2
- removed link little_link3
- removed link little_link4
- removed link middle_link0
- removed link middle_link1
- removed link middle_link2
- removed link middle_link3
- removed link middle_link4
- removed link ring_link0
- removed link ring_link1
- removed link ring_link2
- removed link ring_link3
- removed link ring_link4
- removed link thumb_link0
- removed link thumb_link1
- removed link thumb_link2
- removed link thumb_link3
- removed link thumb_link4
- removed link thumb_link5
- added link index_distal, mass 0.00583469729849543; collision mesh filename=meshes/index_distal.STL; visual mesh filename=meshes/index_distal.STL
- added link index_metacarpals, mass 0.00583469729849543; collision mesh filename=meshes/index_metacarpals.STL; visual mesh filename=meshes/index_metacarpals.STL
- added link index_middle, mass 0.00583469729849543; collision mesh filename=meshes/index_middle.STL; visual mesh filename=meshes/index_middle.STL
- added link index_proximal, mass 0.0058347; collision mesh filename=meshes/index_proximal.STL; visual mesh filename=meshes/index_proximal.STL
- added link middle_distal, mass 0.00583469729849543; collision mesh filename=meshes/middle_distal.STL; visual mesh filename=meshes/middle_distal.STL
- added link middle_metacarpals, mass 0.00583469729849543; collision mesh filename=meshes/middle_metacarpals.STL; visual mesh filename=meshes/middle_metacarpals.STL
- added link middle_middle, mass 0.00583469729849543; collision mesh filename=meshes/middle_middle.STL; visual mesh filename=meshes/middle_middle.STL
- added link middle_proximal, mass 0.00583469729849543; collision mesh filename=meshes/middle_proximal.STL; visual mesh filename=meshes/middle_proximal.STL
- added link pinky_distal, mass 0.00583469729849543; collision mesh filename=meshes/pinky_distal.STL; visual mesh filename=meshes/pinky_distal.STL
- added link pinky_metacarpals, mass 0.00583469729849543; collision mesh filename=meshes/pinky_metacarpals.STL; visual mesh filename=meshes/pinky_metacarpals.STL
- added link pinky_middle, mass 0.00583469729849543; collision mesh filename=meshes/pinky_middle.STL; visual mesh filename=meshes/pinky_middle.STL
- added link pinky_proximal, mass 0.00583469729849543; collision mesh filename=meshes/pinky_proximal.STL; visual mesh filename=meshes/pinky_proximal.STL
- added link ring_distal, mass 0.00583469729849543; collision mesh filename=meshes/ring_distal.STL; visual mesh filename=meshes/ring_distal.STL
- added link ring_metacarpals, mass 0.00583469729849543; collision mesh filename=meshes/ring_metacarpals.STL; visual mesh filename=meshes/ring_metacarpals.STL
- added link ring_middle, mass 0.00583469729849543; collision mesh filename=meshes/ring_middle.STL; visual mesh filename=meshes/ring_middle.STL
- added link ring_proximal, mass 0.00583469729849543; collision mesh filename=meshes/ring_proximal.STL; visual mesh filename=meshes/ring_proximal.STL
- added link thumb_distal, mass 0.00583469729849543; collision mesh filename=meshes/thumb_distal.STL; visual mesh filename=meshes/thumb_distal.STL
- added link thumb_metacarpals, mass 0.00583469729849543; collision mesh filename=meshes/thumb_metacarpals.STL; visual mesh filename=meshes/thumb_metacarpals.STL
- added link thumb_metacarpals_base1, mass 0.000117519863807651; collision mesh filename=meshes/thumb_metacarpals_base1.STL; visual mesh filename=meshes/thumb_metacarpals_base1.STL
- added link thumb_metacarpals_base2, mass 0.00583469729849543; collision mesh filename=meshes/thumb_metacarpals_base2.STL; visual mesh filename=meshes/thumb_metacarpals_base2.STL
- added link thumb_proximal, mass 0.00583469729849543; collision mesh filename=meshes/thumb_proximal.STL; visual mesh filename=meshes/thumb_proximal.STL
- link base_link: mass 0.123326285498226 -> 2.91817267018669E-05
Joints:
- removed joint index_joint0
- removed joint index_joint1
- removed joint index_joint2
- removed joint index_joint3
- removed joint index_joint4
- removed joint little_joint0
- removed joint little_joint1
- removed joint little_joint2
- removed joint little_joint3
- removed joint little_joint4
- removed joint middle_joint0
- removed joint middle_joint1
- removed joint middle_joint2
- removed joint middle_joint3
- removed joint middle_joint4
- removed joint ring_joint0
- removed joint ring_joint1
- removed joint ring_joint2
- removed joint ring_joint3
- removed joint ring_joint4
- removed joint thumb_joint0
- removed joint thumb_joint1
- removed joint thumb_joint2
- removed joint thumb_joint3
- removed joint thumb_joint4
- removed joint thumb_joint5
- added joint index_dip: type revolute, parent index_middle, child index_distal, origin xyz=0.00275625762572076 0 0.0317023692875254 rpy=0 -0.217210944617023 0, axis 0 1 0, limit lower=0 upper=1.43 effort=100 velocity=1, mimic joint=index_pip multiplier=0.807909 offset=0
- added joint index_mcp_pitch: type revolute, parent index_metacarpals, child index_proximal, origin xyz=0 0 0 rpy=0 0 0, axis 0 1 0, limit lower=0 upper=1.33 effort=100 velocity=1
- added joint index_mcp_roll: type revolute, parent base_link, child index_metacarpals, origin xyz=-0.0131230356952281 0.0266247663700636 0.159311466218564 rpy=0 0 0, axis 1 0 0, limit lower=-0.18 upper=0.18 effort=100 velocity=1
- added joint index_pip: type revolute, parent index_proximal, child index_middle, origin xyz=-0.00419464197927529 -4.99999969099107E-05 0.0448194271910961 rpy=0 0 0, axis 0 1 0, limit lower=0 upper=1.77 effort=100 velocity=1
- added joint middle_dip: type revolute, parent middle_middle, child middle_distal, origin xyz=0.00275625692744558 0 0.0317023698187573 rpy=0 0 0, axis 0 1 0, limit lower=0 upper=1.43 effort=100 velocity=1, mimic joint=middle_pip multiplier=0.807909 offset=0
- added joint middle_mcp_pitch: type revolute, parent middle_metacarpals, child middle_proximal, origin xyz=0 0 0 rpy=0 0 0, axis 0 1 0, limit lower=0 upper=1.33 effort=100 velocity=1
- added joint middle_mcp_roll: type revolute, parent base_link, child middle_metacarpals, origin xyz=-0.0178568780584143 0.00502476703162374 0.163804355813813 rpy=0 0 0, axis 1 0 0, limit lower=-0.18 upper=0.18 effort=100 velocity=1
- added joint middle_pip: type revolute, parent middle_proximal, child middle_middle, origin xyz=-0.0041946419773943 0 0.0448194271813739 rpy=0 0 0, axis 0 1 0, limit lower=0 upper=1.77 effort=100 velocity=1
- added joint pinky_dip: type revolute, parent pinky_middle, child pinky_distal, origin xyz=0.00275625692744577 0 0.0317023698187571 rpy=0 -0.217210953895726 0, axis 0 1 0, limit lower=0 upper=1.43 effort=100 velocity=1, mimic joint=pinky_pip multiplier=0.807909 offset=0
- added joint pinky_mcp_pitch: type revolute, parent pinky_metacarpals, child pinky_proximal, origin xyz=0 0 0 rpy=0 0 0, axis 0 1 0, limit lower=0 upper=1.33 effort=100 velocity=1
- added joint pinky_mcp_roll: type revolute, parent base_link, child pinky_metacarpals, origin xyz=-0.0119282769782894 -0.0381752349548123 0.150312749584634 rpy=0 0 0, axis 1 0 0, limit lower=-0.18 upper=0.18 effort=100 velocity=1
- added joint pinky_pip: type revolute, parent pinky_proximal, child pinky_middle, origin xyz=-0.00419464197739449 0 0.0448194271912721 rpy=0 0 0, axis 0 1 0, limit lower=0 upper=1.77 effort=100 velocity=1
- added joint ring_dip: type revolute, parent ring_middle, child ring_distal, origin xyz=0.00275625692744577 0 0.0317023698187571 rpy=0 0 0, axis 0 1 0, limit lower=0 upper=1.43 effort=100 velocity=1, mimic joint=ring_pip multiplier=0.807909 offset=0
- added joint ring_mcp_pitch: type revolute, parent ring_metacarpals, child ring_proximal, origin xyz=0 0 0 rpy=0 0 0, axis 0 1 0, limit lower=0 upper=1.33 effort=100 velocity=1
- added joint ring_mcp_roll: type revolute, parent base_link, child ring_metacarpals, origin xyz=-0.0155520472481466 -0.0165752336298738 0.159311470075819 rpy=0 0 0, axis 1 0 0, limit lower=-0.18 upper=0.18 effort=100 velocity=1
- added joint ring_pip: type revolute, parent ring_proximal, child ring_middle, origin xyz=-0.00419464197739421 0 0.044819427181374 rpy=0 0 0, axis 0 1 0, limit lower=0 upper=1.77 effort=100 velocity=1
- added joint thumb_cmc_pitch: type revolute, parent thumb_metacarpals_base2, child thumb_metacarpals, origin xyz=-8.46909131121537E-05 0.0307945044068651 0.00396440678804784 rpy=0 -0.756062553947979 -1.570796326182, axis 0 1 0, limit lower=0 upper=0.6 effort=100 velocity=1
- added joint thumb_cmc_roll: type revolute, parent base_link, child thumb_metacarpals_base1, origin xyz=0.000673424792196536 0.00500849972399572 0.0573919534353699 rpy=0 0 0, axis 0.999999999999929 0 0, limit lower=-0.5 upper=0.8 effort=100 velocity=1
- added joint thumb_cmc_yaw: type revolute, parent thumb_metacarpals_base1, child thumb_metacarpals_base2, origin xyz=0.0229415604675387 0.000833353787679902 0 rpy=0 0 0, axis 0 0 -1, limit lower=0.15 upper=2.2 effort=100 velocity=1
- added joint thumb_ip: type revolute, parent thumb_proximal, child thumb_distal, origin xyz=0.00660276039712052 0 0.0343712870751602 rpy=0 0 0, axis 0 1 0, limit lower=0 upper=1.2 effort=100 velocity=1, mimic joint=thumb_mcp multiplier=1 offset=0
- added joint thumb_mcp: type revolute, parent thumb_metacarpals, child thumb_proximal, origin xyz=0.0040559617361387 0 0.0560833583251174 rpy=0 0 0, axis 0 1 0, limit lower=0 upper=1.2 effort=100 velocity=1
