Commit message: update URDF l20 to v9.0

File: l20/left/linkerhand_l20_left.urdf (robot description, URDF)
Before this commit: robot linkerhand_l20_left.urdf, 22 links, 21 joints
Links:
- link hand_base_link: mass 0.101492069055989 -> 0.101084447002037
- link index_distal: mass 0.00386200107962104 -> 0.00340429158070606
- link index_metacarpals: mass 0.000826416925828409 -> 0.000876740996892305
- link index_middle: mass 0.0018096470933759 -> 0.0024073790765763
- link index_proximal: mass 0.00454034378439372 -> 0.00372419362918456
- link middle_distal: mass 0.00386200248743799 -> 0.00340429126675807
- link middle_metacarpals: mass 0.000826416925828398 -> 0.000876740996892609
- link middle_middle: mass 0.00180964709329765 -> 0.0024073794492107
- link middle_proximal: mass 0.00454034378346624 -> 0.00372419362926555
- link pinky_distal: mass 0.00386200247559812 -> 0.00340429157293531
- link pinky_metacarpals: mass 0.000826416925828368 -> 0.000876740996892322
- link pinky_middle: mass 0.00180964709325975 -> 0.0024073792131766
- link pinky_proximal: mass 0.00454034378334877 -> 0.00372419362915814
- link ring_distal: mass 0.00386200102769892 -> 0.00340429156569409
- link ring_metacarpals: mass 0.000826416925828383 -> 0.000876740996892337
- link ring_middle: mass 0.00180964709329766 -> 0.00240737948314978
- link ring_proximal: mass 0.00454034378337052 -> 0.00372419362925796
- link thumb_distal: mass 0.00432493724895246 -> 0.00408975520701271
- link thumb_metacarpals: mass 0.0120240677638171 -> 0.0229652105738877
- link thumb_metacarpals_base1: mass 0.00274839797669793 -> 0.00459735542885393
- link thumb_metacarpals_base2: mass 0.00427940802750865 -> 0.000997223173061939
- link thumb_proximal: mass 0.00531602156580031 -> 0.00515933884351986
Joints:
- joint index_dip: axis 0 0.999999999999978 0 -> 0 1 0; limit lower=0 upper=1.43 effort=100 velocity=1 -> lower=0 upper=1.4 effort=1 velocity=1; mimic joint=index_pip multiplier=0.807909 offset=0 -> joint=index_pip multiplier=0.8917 offset=0; origin xyz=0.00275581955818074 0 0.0317033719231916 rpy=0 0 0 -> xyz=0.00275561954550102 0 0.0317024252339397 rpy=0 0 0
- joint index_mcp_pitch: axis 0 0.999999999999978 0 -> 0 1 0; limit lower=0 upper=1.33 effort=100 velocity=1 -> lower=0 upper=1.4 effort=1 velocity=1; origin xyz=0.01087006638288 -1.2630433198893E-05 0 rpy=0 0 0 -> xyz=0.0167698082541766 -1.26288306177003E-05 0 rpy=0 0 0
- joint index_mcp_roll: axis 0.999999999999989 0 0 -> 1 0 0; limit lower=-0.18 upper=0.18 effort=100 velocity=1 -> lower=-0.17 upper=0.17 effort=1 velocity=1; origin xyz=-0.0236662629253359 -0.0267021153669649 0.159311473821529 rpy=0 0 0 -> xyz=-0.029865288607565 -0.0266980639200853 0.159311439204817 rpy=0 0 0
- joint index_pip: axis 0 0.999999999999978 0 -> 0 1 0; limit lower=0 upper=1.77 effort=100 velocity=1 -> lower=0 upper=1.57 effort=1 velocity=1; origin xyz=-0.00419480624913221 0 0.0448194128870992 rpy=0 0 0 -> xyz=-0.00419455239160021 0 0.0448194355727413 rpy=0 0 0
- joint middle_dip: axis 0 0.999999999997063 0 -> 0 1 0; limit lower=0 upper=1.43 effort=100 velocity=1 -> lower=0 upper=1.4 effort=1 velocity=1; mimic joint=middle_pip multiplier=0.807909 offset=0 -> joint=middle_pip multiplier=0.8917 offset=0; origin xyz=0.00275581955816206 0 0.0317033719231916 rpy=0 0 0 -> xyz=0.00275561954550102 0 0.0317024252339387 rpy=0 0 0
- joint middle_mcp_pitch: axis 0 0.999999999997063 0 -> 0 1 0; limit lower=0 upper=1.33 effort=100 velocity=1 -> lower=0 upper=1.4 effort=1 velocity=1; origin xyz=0.0108700663541581 -1.26551278382542E-05 0 rpy=0 0 0 -> xyz=0.0167698082541766 -1.26288306171729E-05 0 rpy=0 0 0
- joint middle_mcp_roll: axis 0.999999999997074 0 0 -> 1 0 0; limit lower=-0.18 upper=0.18 effort=100 velocity=1 -> lower=-0.17 upper=0.17 effort=1 velocity=1; origin xyz=-0.028550041829013 -0.00510211872877702 0.163804366151529 rpy=0 0 0 -> xyz=-0.0345991283789502 -0.00509806392012034 0.163804328353988 rpy=0 0 0
- joint middle_pip: axis 0 0.999999999997063 0 -> 0 1 0; limit lower=0 upper=1.77 effort=100 velocity=1 -> lower=0 upper=1.57 effort=1 velocity=1; origin xyz=-0.00419480624913501 0 0.0448194128870992 rpy=0 0 0 -> xyz=-0.00419455239160021 0 0.0448194355727413 rpy=0 0 0
- joint pinky_dip: axis 0 0.999999999997607 0 -> 0 1 0; limit lower=0 upper=1.43 effort=100 velocity=1 -> lower=0 upper=1.4 effort=1 velocity=1; mimic joint=pinky_pip multiplier=0.807909 offset=0 -> joint=pinky_pip multiplier=0.8917 offset=0; origin xyz=0.00275581955821799 0 0.0317033719231203 rpy=0 0 0 -> xyz=0.00275561954550002 0 0.0317024252339397 rpy=0 0 0
- joint pinky_mcp_pitch: axis 0 0.999999999997607 0 -> 0 1 0; limit lower=0 upper=1.33 effort=100 velocity=1 -> lower=0 upper=1.4 effort=1 velocity=1; origin xyz=0.0108700663781205 -1.26345288001539E-05 0 rpy=0 0 0 -> xyz=0.0167698082541766 -1.26288306181443E-05 0 rpy=0 0 0
- joint pinky_mcp_roll: axis 0.999999999999863 0 0 -> 1 0 0; limit lower=-0.18 upper=0.18 effort=100 velocity=1 -> lower=-0.17 upper=0.17 effort=1 velocity=1; origin xyz=-0.0226215026189916 0.0380979799565023 0.150312739475098 rpy=0 0 0 -> xyz=-0.0286705351154727 0.0381019360798378 0.150312712339165 rpy=0 0 0
- joint pinky_pip: axis 0 0.999999999997607 0 -> 0 1 0; limit lower=0 upper=1.77 effort=100 velocity=1 -> lower=0 upper=1.57 effort=1 velocity=1; origin xyz=-0.00419480624907856 0 0.0448194128869988 rpy=0 0 0 -> xyz=-0.00419455239160021 0 0.0448194355727413 rpy=0 0 0
- joint ring_dip: axis 0 0.999999999997063 0 -> 0 1 0; limit lower=0 upper=1.43 effort=100 velocity=1 -> lower=0 upper=1.4 effort=1 velocity=1; mimic joint=ring_pip multiplier=0.807909 offset=0 -> joint=ring_pip multiplier=0.8917 offset=0; origin xyz=0.00275581955816206 0 0.0317033719231916 rpy=0 0 0 -> xyz=0.00275561954550363 0 0.0317024242175084 rpy=0 0 0
- joint ring_mcp_pitch: axis 0 0.999999999997063 0 -> 0 1 0; limit lower=0 upper=1.33 effort=100 velocity=1 -> lower=0 upper=1.4 effort=1 velocity=1; origin xyz=0.0108700663541581 -1.26551278382542E-05 0 rpy=0 0 0 -> xyz=0.0167698082541766 -1.26288306177003E-05 0 rpy=0 0 0
- joint ring_mcp_roll: axis 0.999999999997074 0 0 -> 1 0 0; limit lower=-0.18 upper=0.18 effort=100 velocity=1 -> lower=-0.17 upper=0.17 effort=1 velocity=1; origin xyz=-0.026245256656013 0.016497885055223 0.159311479072529 rpy=0 0 0 -> xyz=-0.0322943001717225 0.0165019360798537 0.1593114381003 rpy=0 0 0
- joint ring_pip: axis 0 0.999999999997063 0 -> 0 1 0; limit lower=0 upper=1.77 effort=100 velocity=1 -> lower=0 upper=1.57 effort=1 velocity=1; origin xyz=-0.00419480624913501 0 0.0448194128870992 rpy=0 0 0 -> xyz=-0.00419455239160021 0 0.0448194355727413 rpy=0 0 0
- joint thumb_cmc_pitch: limit lower=0 upper=0.6 effort=100 velocity=1 -> lower=0 upper=0.79 effort=1 velocity=1; origin xyz=0 -0.0307945049899851 0.00396440225285005 rpy=0 -0.767096499588843 1.57079617863246 -> xyz=-0.0011523 -0.00048559 0.030795 rpy=0 0.49978 1.5708; parent thumb_metacarpals_base2 -> thumb_metacarpals_base1
- joint thumb_cmc_roll: axis -0.999999999999989 0 0 -> 0 1 0; limit lower=-0.5 upper=0.8 effort=100 velocity=1 -> lower=0 upper=1.22 effort=1 velocity=1; origin xyz=-0.000566250268316748 -0.00508587816314111 0.0573919459698274 rpy=0 0 0 -> xyz=0.024508 -0.002864 0.0035063 rpy=2.0706 0 0; parent hand_base_link -> thumb_metacarpals_base2
- joint thumb_cmc_yaw: axis 0 0 0.999999999999989 -> -1 0 0; limit lower=0.15 upper=2.2 effort=100 velocity=1 -> lower=0 upper=1.40 effort=1 velocity=1; origin xyz=0.0245077602402008 -0.000833339999216351 0 rpy=0 0 0 -> xyz=-0.00091528 -0.0050818 0.057392 rpy=0 0 0; parent thumb_metacarpals_base1 -> hand_base_link
- joint thumb_ip: limit lower=0 upper=1.2 effort=100 velocity=1 -> lower=0 upper=1.22 effort=1 velocity=1; mimic joint=thumb_mcp multiplier=1 offset=0 -> joint=thumb_mcp multiplier=1.1619 offset=0; origin xyz=-0.00294430789962509 0 0.0344361391557164 rpy=0 0 0 -> xyz=0.0053547 0 0.034485 rpy=0 0 0
- joint thumb_mcp: limit lower=0 upper=1.2 effort=100 velocity=1 -> lower=0 upper=1.05 effort=1 velocity=1; origin xyz=0.00467511679938065 0.00010004081575718 0.0560361883792787 rpy=0 0 0 -> xyz=0.0064539 0 0.055858 rpy=0 0 0

File: l20/right/linkerhand_l20_right.urdf (robot description, URDF)
Before this commit: robot linkerhand_l20_right.urdf, 22 links, 21 joints
Links:
- link base_link: mass 2.91817267018669E-05 -> 0.11937688599385
- link index_distal: mass 0.00583469729849543 -> 0.00337425966618635
- link index_metacarpals: mass 0.00583469729849543 -> 0.000876740424974179
- link index_middle: mass 0.00583469729849543 -> 0.00240726447718958
- link index_proximal: mass 0.0058347 -> 0.00451760211825835
- link middle_distal: mass 0.00583469729849543 -> 0.00337425966615046
- link middle_metacarpals: mass 0.00583469729849543 -> 0.000876740424974166
- link middle_middle: mass 0.00583469729849543 -> 0.00240726449346529
- link middle_proximal: mass 0.00583469729849543 -> 0.00451760211910452
- link pinky_distal: mass 0.00583469729849543 -> 0.00337425966640625
- link pinky_metacarpals: mass 0.00583469729849543 -> 0.000876740424974171
- link pinky_middle: mass 0.00583469729849543 -> 0.00240726454050251
- link pinky_proximal: mass 0.00583469729849543 -> 0.00451760212331234
- link ring_distal: mass 0.00583469729849543 -> 0.00337425966600315
- link ring_metacarpals: mass 0.00583469729849543 -> 0.000876740424974176
- link ring_middle: mass 0.00583469729849543 -> 0.00240726457456344
- link ring_proximal: mass 0.00583469729849543 -> 0.00451760195794046
- link thumb_distal: mass 0.00583469729849543 -> 0.00408969366280382
- link thumb_metacarpals: mass 0.00583469729849543 -> 0.0119766770700791
- link thumb_metacarpals_base1: mass 0.000117519863807651 -> 0.0123205476694916
- link thumb_metacarpals_base2: mass 0.00583469729849543 -> 0.00459772397289602
- link thumb_proximal: mass 0.00583469729849543 -> 0.00515934933952247
Joints:
- removed joint thumb_ip
- added joint thumb_dip: type revolute, parent thumb_proximal, child thumb_distal, origin xyz=0.0066654 0 0.034256 rpy=0 0 0, axis 0 1 0, limit lower=0 upper=1.22 effort=1 velocity=1, mimic joint=thumb_mcp multiplier=1.1619 offset=0
- joint index_dip: limit lower=0 upper=1.43 effort=100 velocity=1 -> lower=0 upper=1.4 effort=1 velocity=1; mimic joint=index_pip multiplier=0.807909 offset=0 -> joint=index_pip multiplier=0.8917 offset=0; origin xyz=0.00275625762572076 0 0.0317023692875254 rpy=0 -0.217210944617023 0 -> xyz=0.00275561951363186 0 0.0317024252223218 rpy=0 0 0
- joint index_mcp_pitch: limit lower=0 upper=1.33 effort=100 velocity=1 -> lower=0 upper=1.4 effort=1 velocity=1; origin xyz=0 0 0 rpy=0 0 0 -> xyz=0.0166748095646496 0 0 rpy=0 0 0
- joint index_mcp_roll: axis 1 0 0 -> 0.999999999998204 0 0; limit lower=-0.18 upper=0.18 effort=100 velocity=1 -> lower=-0.17 upper=0.17 effort=1 velocity=1; origin xyz=-0.0131230356952281 0.0266247663700636 0.159311466218564 rpy=0 0 0 -> xyz=-0.0297703583048348 0.026698113515616 0.159311418025823 rpy=0 0 0
- joint index_pip: limit lower=0 upper=1.77 effort=100 velocity=1 -> lower=0 upper=1.57 effort=1 velocity=1; origin xyz=-0.00419464197927529 -4.99999969099107E-05 0.0448194271910961 rpy=0 0 0 -> xyz=-0.00419455239160021 1.32099983796707E-05 0.0448194355727413 rpy=0 0 0
- joint middle_dip: limit lower=0 upper=1.43 effort=100 velocity=1 -> lower=0 upper=1.4 effort=1 velocity=1; mimic joint=middle_pip multiplier=0.807909 offset=0 -> joint=middle_pip multiplier=0.8917 offset=0; origin xyz=0.00275625692744558 0 0.0317023698187573 rpy=0 0 0 -> xyz=0.00275561956368908 0 0.031702425228504 rpy=0 0 0
- joint middle_mcp_pitch: limit lower=0 upper=1.33 effort=100 velocity=1 -> lower=0 upper=1.4 effort=1 velocity=1; origin xyz=0 0 0 rpy=0 0 0 -> xyz=0.0251050665601614 1.26716622368406E-05 0.00800002169696733 rpy=0 0 0
- joint middle_mcp_roll: axis 1 0 0 -> 0.999999999998204 0 0; limit lower=-0.18 upper=0.18 effort=100 velocity=1 -> lower=-0.17 upper=0.17 effort=1 velocity=1; origin xyz=-0.0178568780584143 0.00502476703162374 0.163804355813813 rpy=0 0 0 -> xyz=-0.0345042006792679 0.00509811417717426 0.163804307612682 rpy=0 0 0
- joint middle_pip: limit lower=0 upper=1.77 effort=100 velocity=1 -> lower=0 upper=1.57 effort=1 velocity=1; origin xyz=-0.0041946419773943 0 0.0448194271813739 rpy=0 0 0 -> xyz=-0.0126248094622216 0 0.0368194524061594 rpy=0 0 0
- joint pinky_dip: limit lower=0 upper=1.43 effort=100 velocity=1 -> lower=0 upper=1.4 effort=1 velocity=1; mimic joint=pinky_pip multiplier=0.807909 offset=0 -> joint=pinky_pip multiplier=0.8917 offset=0; origin xyz=0.00275625692744577 0 0.0317023698187571 rpy=0 -0.217210953895726 0 -> xyz=0.00275561956448663 0 0.0317024252339038 rpy=0 0 0
- joint pinky_mcp_pitch: limit lower=0 upper=1.33 effort=100 velocity=1 -> lower=0 upper=1.4 effort=1 velocity=1; origin xyz=0 0 0 rpy=0 0 0 -> xyz=0.0166748095648401 0 0 rpy=0 0 0
- joint pinky_mcp_roll: axis 1 0 0 -> 0.999999999998204 0 0; limit lower=-0.18 upper=0.18 effort=100 velocity=1 -> lower=-0.17 upper=0.17 effort=1 velocity=1; origin xyz=-0.0119282769782894 -0.0381752349548123 0.150312749584634 rpy=0 0 0 -> xyz=-0.028575599600215 -0.0381024421136991 0.150312739930038 rpy=0 0 0
- joint pinky_pip: limit lower=0 upper=1.77 effort=100 velocity=1 -> lower=0 upper=1.57 effort=1 velocity=1; origin xyz=-0.00419464197739449 0 0.0448194271912721 rpy=0 0 0 -> xyz=-0.00419455244191127 1.32099958100595E-05 0.0448194355633776 rpy=0 0 0
- joint ring_dip: limit lower=0 upper=1.43 effort=100 velocity=1 -> lower=0 upper=1.4 effort=1 velocity=1; mimic joint=ring_pip multiplier=0.807909 offset=0 -> joint=ring_pip multiplier=0.8917 offset=0; origin xyz=0.00275625692744577 0 0.0317023698187571 rpy=0 0 0 -> xyz=0.00275561956405355 0 0.0317024252327154 rpy=0 0 0
- joint ring_mcp_pitch: limit lower=0 upper=1.33 effort=100 velocity=1 -> lower=0 upper=1.4 effort=1 velocity=1; origin xyz=0 0 0 rpy=0 0 0 -> xyz=0.0251050665600563 1.26716622367851E-05 0.00800002169746956 rpy=0 0 0
- joint ring_mcp_roll: axis 1 0 0 -> 0.999999999998204 0 0; limit lower=-0.18 upper=0.18 effort=100 velocity=1 -> lower=-0.17 upper=0.17 effort=1 velocity=1; origin xyz=-0.0155520472481466 -0.0165752336298738 0.159311470075819 rpy=0 0 0 -> xyz=-0.0321993698689908 -0.0165018864843229 0.159311421874683 rpy=0 0 0
- joint ring_pip: limit lower=0 upper=1.77 effort=100 velocity=1 -> lower=0 upper=1.57 effort=1 velocity=1; origin xyz=-0.00419464197739421 0 0.044819427181374 rpy=0 0 0 -> xyz=-0.0126248094619703 0 0.0368194524036704 rpy=0 0 0
- joint thumb_cmc_pitch: limit lower=0 upper=0.6 effort=100 velocity=1 -> lower=0 upper=0.79 effort=1 velocity=1; origin xyz=-8.46909131121537E-05 0.0307945044068651 0.00396440678804784 rpy=0 -0.756062553947979 -1.570796326182 -> xyz=-0.00010969 -0.0039644 0.030795 rpy=0 0.38815 -1.5708
- joint thumb_cmc_roll: axis 0.999999999999929 0 0 -> 0 1 0; child thumb_metacarpals_base1 -> thumb_metacarpals_base2; limit lower=-0.5 upper=0.8 effort=100 velocity=1 -> lower=0 upper=1.22 effort=1 velocity=1; origin xyz=0.000673424792196536 0.00500849972399572 0.0573919534353699 rpy=0 0 0 -> xyz=0.00078474 0.019608 0.00030872 rpy=1.1826 0 1.5708; parent base_link -> thumb_metacarpals_base1
- joint thumb_cmc_yaw: axis 0 0 -1 -> 0 1 0; child thumb_metacarpals_base2 -> thumb_metacarpals_base1; limit lower=0.15 upper=2.2 effort=100 velocity=1 -> lower=0 upper=1.4 effort=1 velocity=1; origin xyz=0.0229415604675387 0.000833353787679902 0 rpy=0 0 0 -> xyz=0.0039847 0.0050818 0.057392 rpy=3.1416 0 1.5708; parent thumb_metacarpals_base1 -> base_link
- joint thumb_mcp: limit lower=0 upper=1.2 effort=100 velocity=1 -> lower=0 upper=1.05 effort=1 velocity=1; origin xyz=0.0040559617361387 0 0.0560833583251174 rpy=0 0 0 -> xyz=0.0085786 0 0.055572 rpy=0 0 0
