Commit message: update o6 urdf

File: o6/left/linkerhand_o6_left.urdf (robot description, URDF)
Before this commit: robot linkerhand_O6_left.urdf, 12 links, 11 joints
Joints:
- joint index_dip: limit lower=0 upper=1.4 effort=100 velocity=1 -> lower=0 upper=1.43 effort=100 velocity=1
- joint index_mcp_pitch: limit lower=0 upper=1.57 effort=100 velocity=1 -> lower=0 upper=1.60 effort=100 velocity=1
- joint middle_dip: limit lower=0 upper=1.4 effort=100 velocity=1 -> lower=0 upper=1.43 effort=100 velocity=1
- joint middle_mcp_pitch: limit lower=0 upper=1.57 effort=100 velocity=1 -> lower=0 upper=1.60 effort=100 velocity=1
- joint pinky_dip: limit lower=0 upper=1.4 effort=100 velocity=1 -> lower=0 upper=1.43 effort=100 velocity=1
- joint pinky_mcp_pitch: limit lower=0 upper=1.57 effort=100 velocity=1 -> lower=0 upper=1.60 effort=100 velocity=1
- joint ring_dip: limit lower=0 upper=1.4 effort=100 velocity=1 -> lower=0 upper=1.43 effort=100 velocity=1
- joint ring_mcp_pitch: limit lower=0 upper=1.57 effort=100 velocity=1 -> lower=0 upper=1.60 effort=100 velocity=1
- joint thumb_cmc_pitch: limit lower=0 upper=0.52 effort=100 velocity=1 -> lower=0 upper=0.58 effort=100 velocity=1
- joint thumb_cmc_yaw: limit lower=0 upper=1.54 effort=100 velocity=1 -> lower=0 upper=1.36 effort=100 velocity=1
- joint thumb_ip: limit lower=0 upper=0.96 effort=100 velocity=1 -> lower=0 upper=1.08 effort=100 velocity=1; mimic joint=thumb_cmc_pitch multiplier=1.83 offset=0 -> joint=thumb_cmc_pitch multiplier=1.86 offset=0

File: o6/right/linkerhand_o6_right.urdf (robot description, URDF)
Before this commit: robot linkerhand_O6_right.urdf, 12 links, 11 joints
Joints:
- joint index_dip: limit lower=0 upper=1.4 effort=100 velocity=1 -> lower=0 upper=1.43 effort=100 velocity=1
- joint index_mcp_pitch: limit lower=0 upper=1.57 effort=100 velocity=1 -> lower=0 upper=1.60 effort=100 velocity=1
- joint middle_dip: limit lower=0 upper=1.4 effort=100 velocity=1 -> lower=0 upper=1.43 effort=100 velocity=1
- joint middle_mcp_pitch: limit lower=0 upper=1.57 effort=100 velocity=1 -> lower=0 upper=1.60 effort=100 velocity=1
- joint pinky_dip: limit lower=0 upper=1.4 effort=100 velocity=1 -> lower=0 upper=1.43 effort=100 velocity=1
- joint pinky_mcp_pitch: limit lower=0 upper=1.57 effort=100 velocity=1 -> lower=0 upper=1.60 effort=100 velocity=1
- joint ring_dip: limit lower=0 upper=1.4 effort=100 velocity=1 -> lower=0 upper=1.43 effort=100 velocity=1
- joint ring_mcp_pitch: limit lower=0 upper=1.57 effort=100 velocity=1 -> lower=0 upper=1.60 effort=100 velocity=1
- joint thumb_cmc_pitch: limit lower=0 upper=0.52 effort=100 velocity=1 -> lower=0 upper=0.58 effort=100 velocity=1
- joint thumb_cmc_yaw: limit lower=0 upper=1.54 effort=100 velocity=1 -> lower=0 upper=1.36 effort=100 velocity=1
- joint thumb_ip: limit lower=0 upper=0.96 effort=100 velocity=1 -> lower=0 upper=1.08 effort=100 velocity=1; mimic joint=thumb_cmc_pitch multiplier=1.83 offset=0 -> joint=thumb_cmc_pitch multiplier=1.86 offset=0

Commit message: Update thumb joint coupling and abduction–adduction limits

File: o6/left/linkerhand_o6_left.urdf (robot description, URDF)
Before this commit: robot linker_o6_left_v1.0_urdf, 12 links, 11 joints
Joints:
- joint thumb_cmc_yaw: limit lower=0 upper=1.36 effort=100 velocity=1 -> lower=0 upper=1.3 effort=100 velocity=1
- joint thumb_ip: mimic joint=thumb_cmc_pitch multiplier=1.86 offset=0 -> joint=thumb_cmc_pitch multiplier=2.29 offset=0
