Commit message: update l20 right urdf

File: l20/right/linkerhand_l20_right.urdf (robot description, URDF)
Before this commit: robot linker_l20_right_v9.0_urdf, 22 links, 21 joints
Links:
- link base_link: mass 0.11937688599385 -> 0.119355521222427
- link index_distal: mass 0.00337425966618635 -> 0.0033741266988187
- link index_metacarpals: mass 0.000876740424974179 -> 0.000876738307234888
- link index_middle: mass 0.00240726447718958 -> 0.00240742140798158
- link index_proximal: mass 0.00451760211825835 -> 0.00451758879934099
- link middle_distal: mass 0.00337425966615046 -> 0.00337412669879527
- link middle_metacarpals: mass 0.000876740424974166 -> 0.000876738307234834
- link middle_middle: mass 0.00240726449346529 -> 0.00240742140799016
- link middle_proximal: mass 0.00451760211910452 -> 0.00451758879836063
- link pinky_distal: mass 0.00337425966640625 -> 0.00337412669848792
- link pinky_metacarpals: mass 0.000876740424974171 -> 0.000876738307234833
- link pinky_middle: mass 0.00240726454050251 -> 0.00240742140800545
- link pinky_proximal: mass 0.00451760212331234 -> 0.00451758867960127
- link ring_distal: mass 0.00337425966600315 -> 0.0033741266986076
- link ring_metacarpals: mass 0.000876740424974176 -> 0.000876738307234883
- link ring_middle: mass 0.00240726457456344 -> 0.00240742140052362
- link ring_proximal: mass 0.00451760195794046 -> 0.00451758885102983
- link thumb_distal: mass 0.00408969366280382 -> 0.00614449456083594
- link thumb_metacarpals: mass 0.0119766770700791 -> 0.0119728760675928
- link thumb_metacarpals_base1: mass 0.0123205476694916 -> 0.0123197273270212
- link thumb_metacarpals_base2: mass 0.00459772397289602 -> 0.00459776097124383
- link thumb_proximal: mass 0.00515934933952247 -> 0.00515940162015082
Joints:
- joint middle_mcp_pitch: origin xyz=0.0251050665601614 1.26716622368406E-05 0.00800002169696733 rpy=0 0 0 -> xyz=0.0166748095398548 1.26556862705962E-05 0 rpy=0 0 0
- joint middle_pip: origin xyz=-0.0126248094622216 0 0.0368194524061594 rpy=0 0 0 -> xyz=-0.00419455244189623 0 0.0448194355665477 rpy=0 0 0
- joint pinky_dip: origin xyz=0.00275561956448663 0 0.0317024252339038 rpy=0 0 0 -> xyz=0.0027556 0 0.031702 rpy=0 0 0
- joint pinky_mcp_pitch: origin xyz=0.0166748095648401 0 0 rpy=0 0 0 -> xyz=0.016675 0 0 rpy=0 0 0
- joint pinky_mcp_roll: axis 0.999999999998204 0 0 -> 1 0 0; origin xyz=-0.028575599600215 -0.0381024421136991 0.150312739930038 rpy=0 0 0 -> xyz=-0.028576 -0.038102 0.15031 rpy=0 0 0
- joint ring_mcp_pitch: origin xyz=0.0251050665600563 1.26716622367851E-05 0.00800002169746956 rpy=0 0 0 -> xyz=0.016675 1.2656E-05 0 rpy=0 0 0
- joint ring_mcp_roll: axis 0.999999999998204 0 0 -> 1 0 0; origin xyz=-0.0321993698689908 -0.0165018864843229 0.159311421874683 rpy=0 0 0 -> xyz=-0.032199 -0.016502 0.15931 rpy=0 0 0
- joint ring_pip: origin xyz=-0.0126248094619703 0 0.0368194524036704 rpy=0 0 0 -> xyz=-0.00419455244174995 0 0.0448194355645609 rpy=0 0 0
- joint thumb_cmc_pitch: origin xyz=-0.00010969 -0.0039644 0.030795 rpy=0 0.38815 -1.5708 -> xyz=-0.000109690908352875 -0.00396440679180957 0.0307945044045898 rpy=0 0.388152995607441 -1.57079632624948
- joint thumb_cmc_roll: origin xyz=0.00078474 0.019608 0.00030872 rpy=1.1826 0 1.5708 -> xyz=0.000784740002368223 0.0196077603627024 0.000308721957079858 rpy=1.18264333118745 0 1.57079632679503
- joint thumb_dip: origin xyz=0.0066654 0 0.034256 rpy=0 0 0 -> xyz=0.0066653832125308 0 0.0342561774516276 rpy=0 0 0
- joint thumb_mcp: origin xyz=0.0085786 0 0.055572 rpy=0 0 0 -> xyz=0.00857856380171737 0 0.0555715948082196 rpy=0 0 0
