Commit message: Add urdf o6/l6

File: l6/left/linkerhand_l6_left.urdf (robot description, URDF)
Before this commit: robot linkerhand_O6_right.urdf, 12 links, 11 joints
Links:
- removed link thumb_metacarpals_base2
- added link thumb_metacarpals_base1, mass 0.989011744524491; collision mesh filename=meshes/thumb_metacarpals_base1.STL; visual mesh filename=meshes/thumb_metacarpals_base1.STL
- link hand_base_link: mass 0.06740077960995 -> 0.989011744524491
- link index_distal: mass 0.00376787129082313 -> 0.989011744524491
- link index_proximal: mass 0.00253178529301663 -> 0.989011744524491
- link middle_distal: mass 0.00376786259758948 -> 0.989011744524491
- link middle_proximal: mass 0.00253175497594429 -> 0.989011744524491
- link pinky_distal: mass 0.00376782669873412 -> 0.989011744524491
- link pinky_proximal: mass 0.00253167400540778 -> 0.989011744524491
- link ring_distal: mass 0.0037678395356105 -> 0.989011744524491
- link ring_proximal: mass 0.00253170963529411 -> 0.989011744524491
- link thumb_distal: mass 0.00763302603723749 -> 0.989011744524491
- link thumb_metacarpals: mass 0.0123381607727595 -> 0.989011744524491
Joints:
- removed joint thumb_cmc_yaw
- removed joint thumb_ip
- added joint thumb_dip: type revolute, parent thumb_metacarpals, child thumb_distal, origin xyz=0 0.0061 0.0827 rpy=0.33787 0 0, axis -1 0 0, limit lower=0 upper=1.22 effort=0 velocity=0, mimic joint=thumb_cmc_pitch multiplier=2.22 offset=0
- added joint thunb_cmc_roll: type revolute, parent hand_base_link, child thumb_metacarpals_base1, origin xyz=0.0078133 -0.029898 0.026692 rpy=-0.034907 0 0, axis 0 0 1, limit lower=0 upper=1.39 effort=0 velocity=0
- joint index_dip: limit lower=0 upper=1.4 effort=100 velocity=1 -> lower=0 upper=1.14 effort=0 velocity=0; mimic joint=index_mcp_pitch multiplier=0.89 offset=0 -> joint=index_mcp_pitch multiplier=1.9 offset=0; origin xyz=-0.0052516 0 0.036625 rpy=0 0 0 -> xyz=0.00093749 0 0.028002 rpy=0 0 0
- joint index_mcp_pitch: limit lower=0 upper=1.57 effort=100 velocity=1 -> lower=0 upper=1.26 effort=0 velocity=0; origin xyz=0.0024758 0.02419 0.098779 rpy=-0.05236 0 0 -> xyz=-0.00066821 -0.028834 0.12104 rpy=0.05236 0 0
- joint middle_dip: limit lower=0 upper=1.4 effort=100 velocity=1 -> lower=0 upper=1.14 effort=0 velocity=0; mimic joint=middle_mcp_pitch multiplier=0.89 offset=0 -> joint=middle_mcp_pitch multiplier=1.9 offset=0; origin xyz=-0.0052516 0 0.036625 rpy=0 0 0 -> xyz=0.00093749 0 0.028002 rpy=0 0 0
- joint middle_mcp_pitch: limit lower=0 upper=1.57 effort=100 velocity=1 -> lower=0 upper=1.26 effort=0 velocity=0; origin xyz=0.00052576 0.00634 0.1027 rpy=0 0 0 -> xyz=-0.00066821 -0.0087679 0.12704 rpy=0 0 0
- joint pinky_dip: limit lower=0 upper=1.4 effort=100 velocity=1 -> lower=0 upper=1.14 effort=0 velocity=0; mimic joint=pinky_mcp_pitch multiplier=0.89 offset=0 -> joint=pinky_mcp_pitch multiplier=1.9 offset=0; origin xyz=-0.0052516 0 0.036625 rpy=0 0 0 -> xyz=0.00093723 0 0.028002 rpy=0 0 0
- joint pinky_mcp_pitch: limit lower=0 upper=1.57 effort=100 velocity=1 -> lower=0 upper=1.26 effort=0 velocity=0; origin xyz=0.0024758 -0.028372 0.092741 rpy=0.087266 0 0 -> xyz=-0.00067852 0.029947 0.11806 rpy=-0.087266 0 0
- joint ring_dip: limit lower=0 upper=1.4 effort=100 velocity=1 -> lower=0 upper=1.14 effort=0 velocity=0; mimic joint=ring_mcp_pitch multiplier=0.89 offset=0 -> joint=ring_mcp_pitch multiplier=1.9 offset=0; origin xyz=-0.0052516 0 0.036625 rpy=0 0 0 -> xyz=0.00093723 0 0.028002 rpy=0 0 0
- joint ring_mcp_pitch: limit lower=0 upper=1.57 effort=100 velocity=1 -> lower=0 upper=1.26 effort=0 velocity=0; origin xyz=0.0010258 -0.011135 0.098767 rpy=0.05236 0 0 -> xyz=-0.00067368 0.01085 0.12204 rpy=-0.05236 0 0
- joint thumb_cmc_pitch: axis 0 1 0 -> -1 0 0; limit lower=0 upper=0.52 effort=100 velocity=1 -> lower=0 upper=0.99 effort=0 velocity=0; origin xyz=0.0061649 0.010678 -0.004891 rpy=0 -1.1529 -2.0944 -> xyz=0.008374 -0.011838 0.0066685 rpy=1.2615 0 0.61087; parent thumb_metacarpals_base2 -> thumb_metacarpals_base1

File: l6/right/linkerhand_l6_right.urdf (robot description, URDF)
Before this commit: robot linkerhand_O6_right.urdf, 12 links, 11 joints
Links:
- removed link thumb_metacarpals_base2
- added link thumb_metacarpals_base1, mass 0.989012019420379; collision mesh filename=meshes/thumb_metacarpals_base1.STL; visual mesh filename=meshes/thumb_metacarpals_base1.STL
- link hand_base_link: mass 0.06740077960995 -> 0.989012019420379
- link index_distal: mass 0.00376787129082313 -> 0.989012019420379
- link index_proximal: mass 0.00253178529301663 -> 0.989012019420379
- link middle_distal: mass 0.00376786259758948 -> 0.989012019420379
- link middle_proximal: mass 0.00253175497594429 -> 0.989012019420379
- link pinky_distal: mass 0.00376782669873412 -> 0.989012019420379
- link pinky_proximal: mass 0.00253167400540778 -> 0.989012019420379
- link ring_distal: mass 0.0037678395356105 -> 0.989012019420379
- link ring_proximal: mass 0.00253170963529411 -> 0.989012019420379
- link thumb_distal: mass 0.00763302603723749 -> 0.989012019420379
- link thumb_metacarpals: mass 0.0123381607727595 -> 0.989012019420379
Joints:
- removed joint thumb_cmc_yaw
- added joint thunb_cmc_roll: type revolute, parent hand_base_link, child thumb_metacarpals_base1, origin xyz=0.0078133 0.030812 0.025628 rpy=0 0 0, axis 0 0 -1, limit lower=0 upper=1.39 effort=0 velocity=0
- joint index_dip: limit lower=0 upper=1.4 effort=100 velocity=1 -> lower=0 upper=1.14 effort=0 velocity=0; mimic joint=index_mcp_pitch multiplier=0.89 offset=0 -> joint=index_mcp_pitch multiplier=1.9 offset=0; origin xyz=-0.0052516 0 0.036625 rpy=0 0 0 -> xyz=0.0012095 0 0.027992 rpy=0 0 0
- joint index_mcp_pitch: limit lower=0 upper=1.57 effort=100 velocity=1 -> lower=0 upper=1.26 effort=0 velocity=0; origin xyz=0.0024758 0.02419 0.098779 rpy=-0.05236 0 0 -> xyz=-0.00066821 0.033041 0.11614 rpy=-0.087266 0 0
- joint middle_dip: limit lower=0 upper=1.4 effort=100 velocity=1 -> lower=0 upper=1.14 effort=0 velocity=0; mimic joint=middle_mcp_pitch multiplier=0.89 offset=0 -> joint=middle_mcp_pitch multiplier=1.9 offset=0; origin xyz=-0.0052516 0 0.036625 rpy=0 0 0 -> xyz=0.0009359 0 0.028002 rpy=0 0 0
- joint middle_mcp_pitch: limit lower=0 upper=1.57 effort=100 velocity=1 -> lower=0 upper=1.26 effort=0 velocity=0; origin xyz=0.00052576 0.00634 0.1027 rpy=0 0 0 -> xyz=-0.00066821 0.013196 0.12284 rpy=-0.034907 0 0
- joint pinky_dip: axis 0 1 0 -> 0.00010331 1 0; limit lower=0 upper=1.4 effort=100 velocity=1 -> lower=0 upper=1.14 effort=0 velocity=0; mimic joint=pinky_mcp_pitch multiplier=0.89 offset=0 -> joint=pinky_mcp_pitch multiplier=1.9 offset=0; origin xyz=-0.0052516 0 0.036625 rpy=0 0 0 -> xyz=0.0009359 0 0.028002 rpy=0 0 0
- joint pinky_mcp_pitch: axis 0 1 0 -> -0.00010331 1 0; limit lower=0 upper=1.57 effort=100 velocity=1 -> lower=0 upper=1.26 effort=0 velocity=0; origin xyz=0.0024758 -0.028372 0.092741 rpy=0.087266 0 0 -> xyz=-0.00067852 -0.025809 0.11521 rpy=0.05236 0 -0.00010364
- joint ring_dip: axis 0 1 0 -> 0.00017246 1 0; limit lower=0 upper=1.4 effort=100 velocity=1 -> lower=0 upper=1.14 effort=0 velocity=0; mimic joint=ring_mcp_pitch multiplier=0.89 offset=0 -> joint=ring_mcp_pitch multiplier=1.9 offset=0; origin xyz=-0.0052516 0 0.036625 rpy=0 0 0 -> xyz=0.0009359 0 0.028002 rpy=0 0 0
- joint ring_mcp_pitch: axis 0 1 0 -> -0.00017246 1 0; limit lower=0 upper=1.57 effort=100 velocity=1 -> lower=0 upper=1.26 effort=0 velocity=0; origin xyz=0.0010258 -0.011135 0.098767 rpy=0.05236 0 0 -> xyz=-0.00067368 -0.0065844 0.11852 rpy=0.017453 0 -0.00017259
- joint thumb_cmc_pitch: axis 0 1 0 -> 1 0 0; limit lower=0 upper=0.52 effort=100 velocity=1 -> lower=0 upper=0.99 effort=0 velocity=0; origin xyz=0.0061649 0.010678 -0.004891 rpy=0 -1.1529 -2.0944 -> xyz=0.0081692 0.011981 0.00275 rpy=-1.4249 0 -0.61087; parent thumb_metacarpals_base2 -> thumb_metacarpals_base1
- joint thumb_ip: axis 0 1 0 -> 1 0 0; limit lower=0 upper=0.96 effort=100 velocity=1 -> lower=0 upper=1.22 effort=0 velocity=0; mimic joint=thumb_cmc_pitch multiplier=1.83 offset=0 -> joint=thumb_cmc_pitch multiplier=2.22 offset=0; origin xyz=0.0037776 0 0.045368 rpy=0 0 0 -> xyz=0 -0.0061 0.0827 rpy=0 0 0

File: o6/left/linkerhand_o6_left.urdf (robot description, URDF)
Before this commit: robot linkerhand_O6_left.urdf, 12 links, 11 joints
Joints:
- joint index_dip: limit lower=0 upper=1.43 effort=100 velocity=1 -> lower=0 upper=1.4 effort=100 velocity=1
- joint index_mcp_pitch: limit lower=0 upper=1.60 effort=100 velocity=1 -> lower=0 upper=1.57 effort=100 velocity=1
- joint middle_dip: limit lower=0 upper=1.43 effort=100 velocity=1 -> lower=0 upper=1.4 effort=100 velocity=1
- joint middle_mcp_pitch: limit lower=0 upper=1.60 effort=100 velocity=1 -> lower=0 upper=1.57 effort=100 velocity=1
- joint pinky_dip: limit lower=0 upper=1.43 effort=100 velocity=1 -> lower=0 upper=1.4 effort=100 velocity=1
- joint pinky_mcp_pitch: limit lower=0 upper=1.60 effort=100 velocity=1 -> lower=0 upper=1.57 effort=100 velocity=1
- joint ring_dip: limit lower=0 upper=1.43 effort=100 velocity=1 -> lower=0 upper=1.4 effort=100 velocity=1
- joint ring_mcp_pitch: limit lower=0 upper=1.60 effort=100 velocity=1 -> lower=0 upper=1.57 effort=100 velocity=1
- joint thumb_cmc_pitch: limit lower=0 upper=0.58 effort=100 velocity=1 -> lower=0 upper=0.52 effort=100 velocity=1
- joint thumb_cmc_yaw: limit lower=0 upper=1.36 effort=100 velocity=1 -> lower=0 upper=1.54 effort=100 velocity=1
- joint thumb_ip: limit lower=0 upper=1.08 effort=100 velocity=1 -> lower=0 upper=0.96 effort=100 velocity=1; mimic joint=thumb_cmc_pitch multiplier=1.86 offset=0 -> joint=thumb_cmc_pitch multiplier=1.83 offset=0

Commit message: update l6 left&right urdf

File: l6/left/linkerhand_l6_left.urdf (robot description, URDF)
Before this commit: robot linkerhand_L6_left, 12 links, 11 joints
Joints:
- joint pinky_dip: origin xyz=0.00093723 0 0.028002 rpy=0 0 0 -> xyz=0.00093723 0.0049277 0.028002 rpy=0 0 0
- joint pinky_mcp_pitch: origin xyz=-0.00067852 0.029947 0.11806 rpy=-0.087266 0 0 -> xyz=-0.00067852 0.025038 0.11849 rpy=-0.087266 0 0
- joint thumb_cmc_pitch: origin xyz=0.008374 -0.011838 0.0066685 rpy=1.2615 0 0.61087 -> xyz=0.0050248 -0.013602 0.0066685 rpy=1.2615 0 0.34907
- joint thumb_dip: origin xyz=0 0.0061 0.0827 rpy=0.33787 0 0 -> xyz=0 0.0061 0.0827 rpy=0.34208 0 0

File: l6/right/linkerhand_l6_right.urdf (robot description, URDF)
Before this commit: robot linkerhand_L6_right, 12 links, 11 joints
Joints:
- removed joint thumb_ip
- added joint thumb_dip: type revolute, parent thumb_metacarpals, child thumb_distal, origin xyz=0 -0.0061 0.0827 rpy=0 0 0, axis 1 0 0, limit lower=0 upper=1.22 effort=0 velocity=0, mimic joint=thumb_cmc_pitch multiplier=2.22 offset=0
- joint pinky_dip: axis 0.00010331 1 0 -> 0 1 0
- joint pinky_mcp_pitch: axis -0.00010331 1 0 -> 0 1 0
- joint ring_dip: axis 0.00017246 1 0 -> 0 1 0
- joint ring_mcp_pitch: axis -0.00017246 1 0 -> 0 1 0
- joint thunb_cmc_roll: axis 0 0 -1 -> 0 0 1; limit lower=0 upper=1.39 effort=0 velocity=0 -> lower=-1.39 upper=0 effort=0 velocity=0
