Commit message: Updated L6 URDF version number to 2.1 to keep everything consistent. Fixed all PR comment suggestions

File: l6/left/linkerhand_L6V3.1_left.urdf (robot description, URDF)
Before this commit: robot linkerhand_L6V3.1_left_1.9, 12 links, 11 joints
Links:
- removed link hand_base_link
- removed link index_distal
- removed link index_proximal
- removed link middle_distal
- removed link middle_proximal
- removed link pinky_distal
- removed link pinky_proximal
- removed link ring_distal
- removed link ring_proximal
- removed link thumb_distal
- removed link thumb_metacarpals
- removed link thumb_metacarpals_base1
- added link lh_hand_base_link, mass 0.4185; collision mesh filename=meshes/hand_base_link.STL; visual mesh filename=meshes/hand_base_link.STL
- added link lh_index_distal, mass 0.018408; collision mesh filename=meshes/index_distal.STL; visual mesh filename=meshes/index_distal.STL
- added link lh_index_proximal, mass 0.008553; collision mesh filename=meshes/index_proximal.STL; visual mesh filename=meshes/index_proximal.STL
- added link lh_middle_distal, mass 0.018408; collision mesh filename=meshes/middle_distal.STL; visual mesh filename=meshes/middle_distal.STL
- added link lh_middle_proximal, mass 0.008553; collision mesh filename=meshes/middle_proximal.STL; visual mesh filename=meshes/middle_proximal.STL
- added link lh_pinky_distal, mass 0.018408; collision mesh filename=meshes/pinky_distal.STL; visual mesh filename=meshes/pinky_distal.STL
- added link lh_pinky_proximal, mass 0.008553; collision mesh filename=meshes/pinky_proximal.STL; visual mesh filename=meshes/pinky_proximal.STL
- added link lh_ring_distal, mass 0.018408; collision mesh filename=meshes/ring_distal.STL; visual mesh filename=meshes/ring_distal.STL
- added link lh_ring_proximal, mass 0.008553; collision mesh filename=meshes/ring_proximal.STL; visual mesh filename=meshes/ring_proximal.STL
- added link lh_thumb_distal, mass 0.018; collision mesh filename=meshes/thumb_distal.STL; visual mesh filename=meshes/thumb_distal.STL
- added link lh_thumb_metacarpals, mass 0.065; collision mesh filename=meshes/thumb_metacarpals.STL; visual mesh filename=meshes/thumb_metacarpals.STL
- added link lh_thumb_metacarpals_base1, mass 0.01; collision mesh filename=meshes/thumb_metacarpals_base1.STL; visual mesh filename=meshes/thumb_metacarpals_base1.STL
Joints:
- removed joint index_dip
- removed joint index_mcp_pitch
- removed joint middle_dip
- removed joint middle_mcp_pitch
- removed joint pinky_dip
- removed joint pinky_mcp_pitch
- removed joint ring_dip
- removed joint ring_mcp_pitch
- removed joint thumb_cmc_pitch
- removed joint thumb_cmc_roll
- removed joint thumb_dip
- added joint lh_index_dip: type revolute, parent lh_index_proximal, child lh_index_distal, origin xyz=0.001001 -0.000537 0.028003 rpy=0 0 0, axis 0 1 0, limit lower=0 upper=1.277039 effort=0 velocity=3.1, mimic joint=lh_index_mcp_pitch multiplier=1.125676 offset=0
- added joint lh_index_mcp_pitch: type revolute, parent lh_hand_base_link, child lh_index_proximal, origin xyz=-0.00066821 -0.028967 0.11722 rpy=0 0 0, axis 0 1 0, limit lower=0 upper=1.134464 effort=0.574 velocity=6.10
- added joint lh_middle_dip: type revolute, parent lh_middle_proximal, child lh_middle_distal, origin xyz=0.000994 0.000058 0.028008 rpy=0 0 0, axis 0 1 0, limit lower=0 upper=1.277039 effort=0 velocity=3.1, mimic joint=lh_middle_mcp_pitch multiplier=1.125676 offset=0
- added joint lh_middle_mcp_pitch: type revolute, parent lh_hand_base_link, child lh_middle_proximal, origin xyz=-0.00066821 -0.0089013 0.12322 rpy=0 0 0, axis 0 1 0, limit lower=0 upper=1.134464 effort=0.574 velocity=6.10
- added joint lh_pinky_dip: type revolute, parent lh_pinky_proximal, child lh_pinky_distal, origin xyz=0.000979 0.001534 0.027967 rpy=0 0 0, axis 0 1 0, limit lower=0 upper=1.277039 effort=0 velocity=3.1, mimic joint=lh_pinky_mcp_pitch multiplier=1.125676 offset=0
- added joint lh_pinky_mcp_pitch: type revolute, parent lh_hand_base_link, child lh_pinky_proximal, origin xyz=-0.00067852 0.029814 0.11424 rpy=0 0 0, axis 0 1 0, limit lower=0 upper=1.134464 effort=0.574 velocity=6.10
- added joint lh_ring_dip: type revolute, parent lh_ring_proximal, child lh_ring_distal, origin xyz=0.000979 0.001534 0.027967 rpy=0 0 0, axis 0 1 0, limit lower=0 upper=1.277039 effort=0 velocity=3.1, mimic joint=lh_ring_mcp_pitch multiplier=1.125676 offset=0
- added joint lh_ring_mcp_pitch: type revolute, parent lh_hand_base_link, child lh_ring_proximal, origin xyz=-0.00067368 0.010717 0.11822 rpy=0 0 0, axis 0 1 0, limit lower=0 upper=1.134464 effort=0.574 velocity=6.10
- added joint lh_thumb_cmc_pitch: type revolute, parent lh_thumb_metacarpals_base1, child lh_thumb_metacarpals, origin xyz=0.0057298 -0.01332 0.0027456 rpy=1.1083 0 0.40143, axis -1 0 0, limit lower=0 upper=0.837758 effort=1.008 velocity=3.47
- added joint lh_thumb_cmc_roll: type revolute, parent lh_hand_base_link, child lh_thumb_metacarpals_base1, origin xyz=0.0078133 -0.029898 0.026692 rpy=-0.034907 0 0, axis 0 0 1, limit lower=-0.087266 upper=1.256637 effort=0.588 velocity=5.95
- added joint lh_thumb_dip: type revolute, parent lh_thumb_metacarpals, child lh_thumb_distal, origin xyz=0 0.0061 0.0827 rpy=0 0 0, axis -1 0 0, limit lower=0 upper=0.963287 effort=0 velocity=1.7, mimic joint=lh_thumb_cmc_pitch multiplier=1.226495 offset=0

File: l6/right/linkerhand_L6V3.1_right.urdf (robot description, URDF)
Before this commit: robot linkerhand_L6V3.1_right_3.3, 12 links, 11 joints
Links:
- removed link hand_base_link
- removed link index_distal
- removed link index_proximal
- removed link middle_distal
- removed link middle_proximal
- removed link pinky_distal
- removed link pinky_proximal
- removed link ring_distal
- removed link ring_proximal
- removed link thumb_distal
- removed link thumb_metacarpals
- removed link thumb_metacarpals_base1
- added link rh_hand_base_link, mass 0.4185; collision mesh filename=meshes/hand_base_link.STL; visual mesh filename=meshes/hand_base_link.STL
- added link rh_index_distal, mass 0.018408; collision mesh filename=meshes/index_distal.STL; visual mesh filename=meshes/index_distal.STL
- added link rh_index_proximal, mass 0.008553; collision mesh filename=meshes/index_proximal.STL; visual mesh filename=meshes/index_proximal.STL
- added link rh_middle_distal, mass 0.018408; collision mesh filename=meshes/middle_distal.STL; visual mesh filename=meshes/middle_distal.STL
- added link rh_middle_proximal, mass 0.008553; collision mesh filename=meshes/middle_proximal.STL; visual mesh filename=meshes/middle_proximal.STL
- added link rh_pinky_distal, mass 0.018408; collision mesh filename=meshes/pinky_distal.STL; visual mesh filename=meshes/pinky_distal.STL
- added link rh_pinky_proximal, mass 0.008553; collision mesh filename=meshes/pinky_proximal.STL; visual mesh filename=meshes/pinky_proximal.STL
- added link rh_ring_distal, mass 0.018408; collision mesh filename=meshes/ring_distal.STL; visual mesh filename=meshes/ring_distal.STL
- added link rh_ring_proximal, mass 0.008553; collision mesh filename=meshes/ring_proximal.STL; visual mesh filename=meshes/ring_proximal.STL
- added link rh_thumb_distal, mass 0.018; collision mesh filename=meshes/thumb_distal.STL; visual mesh filename=meshes/thumb_distal.STL
- added link rh_thumb_metacarpals, mass 0.065; collision mesh filename=meshes/thumb_metacarpals.STL; visual mesh filename=meshes/thumb_metacarpals.STL
- added link rh_thumb_metacarpals_base1, mass 0.01; collision mesh filename=meshes/thumb_metacarpals_base1.STL; visual mesh filename=meshes/thumb_metacarpals_base1.STL
Joints:
- removed joint index_dip
- removed joint index_mcp_pitch
- removed joint middle_dip
- removed joint middle_mcp_pitch
- removed joint pinky_dip
- removed joint pinky_mcp_pitch
- removed joint ring_dip
- removed joint ring_mcp_pitch
- removed joint thumb_cmc_pitch
- removed joint thumb_cmc_roll
- removed joint thumb_dip
- added joint rh_index_dip: type revolute, parent rh_index_proximal, child rh_index_distal, origin xyz=0.0009359 0 0.028002 rpy=0 0 0, axis 0 1 0, limit lower=0 upper=1.277039 effort=0 velocity=3.1, mimic joint=rh_index_mcp_pitch multiplier=1.125676 offset=0
- added joint rh_index_mcp_pitch: type revolute, parent rh_hand_base_link, child rh_index_proximal, origin xyz=-0.00066821 0.033467 0.11622 rpy=-0.087266 0 0, axis 0 1 0, limit lower=0 upper=1.134464 effort=0.574 velocity=6.10
- added joint rh_middle_dip: type revolute, parent rh_middle_proximal, child rh_middle_distal, origin xyz=0.0009359 0 0.028002 rpy=0 0 0, axis 0 1 0, limit lower=0 upper=1.277039 effort=0 velocity=3.1, mimic joint=rh_middle_mcp_pitch multiplier=1.125676 offset=0
- added joint rh_middle_mcp_pitch: type revolute, parent rh_hand_base_link, child rh_middle_proximal, origin xyz=-0.00066821 0.0134013 0.12272 rpy=-0.034907 0 0, axis 0 1 0, limit lower=0 upper=1.134464 effort=0.574 velocity=6.10
- added joint rh_pinky_dip: type revolute, parent rh_pinky_proximal, child rh_pinky_distal, origin xyz=0.0009359 0 0.028002 rpy=0 0 0, axis 0 1 0, limit lower=0 upper=1.277039 effort=0 velocity=3.1, mimic joint=rh_pinky_mcp_pitch multiplier=1.125676 offset=0
- added joint rh_pinky_mcp_pitch: type revolute, parent rh_hand_base_link, child rh_pinky_proximal, origin xyz=-0.00067852 -0.025314 0.11474 rpy=0.05236 0 0, axis 0 1 0, limit lower=0 upper=1.134464 effort=0.574 velocity=6.10
- added joint rh_ring_dip: type revolute, parent rh_ring_proximal, child rh_ring_distal, origin xyz=0.0009359 0 0.028002 rpy=0 0 0, axis 0 1 0, limit lower=0 upper=1.277039 effort=0 velocity=3.1, mimic joint=rh_ring_mcp_pitch multiplier=1.125676 offset=0
- added joint rh_ring_mcp_pitch: type revolute, parent rh_hand_base_link, child rh_ring_proximal, origin xyz=-0.00067368 -0.006217 0.11872 rpy=0.017453 0 0, axis 0 1 0, limit lower=0 upper=1.134464 effort=0.574 velocity=6.10
- added joint rh_thumb_cmc_pitch: type revolute, parent rh_thumb_metacarpals_base1, child rh_thumb_metacarpals, origin xyz=0.0054997 0.013314 0.0032166 rpy=-1.0762 0.013637 -0.40121, axis 1 0 0, limit lower=0 upper=0.837758 effort=1.008 velocity=3.47
- added joint rh_thumb_cmc_roll: type revolute, parent rh_hand_base_link, child rh_thumb_metacarpals_base1, origin xyz=0.0078133 0.030812 0.025678 rpy=-0.034907 0 0, axis 0 0.034899 -0.99939, limit lower=-0.087266 upper=1.256637 effort=0.588 velocity=5.95
- added joint rh_thumb_dip: type revolute, parent rh_thumb_metacarpals, child rh_thumb_distal, origin xyz=0 -0.0061 0.0827 rpy=0 0 0, axis 1 0 0, limit lower=0 upper=0.963287 effort=0 velocity=1.7, mimic joint=rh_thumb_cmc_pitch multiplier=1.226495 offset=0

File: o6/left/linkerhand_o6_left.urdf (robot description, URDF)
Before this commit: robot linker_o6_left_v1.0_urdf, 12 links, 11 joints
Links:
- removed link hand_base_link
- removed link index_distal
- removed link index_proximal
- removed link middle_distal
- removed link middle_proximal
- removed link pinky_distal
- removed link pinky_proximal
- removed link ring_distal
- removed link ring_proximal
- removed link thumb_distal
- removed link thumb_metacarpals
- removed link thumb_metacarpals_base2
- added link lh_hand_base_link, mass 0.0672935238166485; collision mesh filename=meshes/hand_base_link.STL; visual mesh filename=meshes/hand_base_link.STL
- added link lh_index_distal, mass 0.00376951085886838; collision mesh filename=meshes/index_distal.STL; visual mesh filename=meshes/index_distal.STL
- added link lh_index_proximal, mass 0.00253174651934627; collision mesh filename=meshes/index_proximal.STL; visual mesh filename=meshes/index_proximal.STL
- added link lh_middle_distal, mass 0.00376952789210256; collision mesh filename=meshes/middle_distal.STL; visual mesh filename=meshes/middle_distal.STL
- added link lh_middle_proximal, mass 0.00253177375206983; collision mesh filename=meshes/middle_proximal.STL; visual mesh filename=meshes/middle_proximal.STL
- added link lh_pinky_distal, mass 0.00376948071276134; collision mesh filename=meshes/pinky_distal.STL; visual mesh filename=meshes/pinky_distal.STL
- added link lh_pinky_proximal, mass 0.00253185993162408; collision mesh filename=meshes/pinky_proximal.STL; visual mesh filename=meshes/pinky_proximal.STL
- added link lh_ring_distal, mass 0.00376949588316609; collision mesh filename=meshes/ring_distal.STL; visual mesh filename=meshes/ring_distal.STL
- added link lh_ring_proximal, mass 0.00253182223645066; collision mesh filename=meshes/ring_proximal.STL; visual mesh filename=meshes/ring_proximal.STL
- added link lh_thumb_distal, mass 0.00763332957284057; collision mesh filename=meshes/thumb_distal.STL; visual mesh filename=meshes/thumb_distal.STL
- added link lh_thumb_metacarpals, mass 0.0123381586619931; collision mesh filename=meshes/thumb_metacarpals.STL; visual mesh filename=meshes/thumb_metacarpals.STL
- added link lh_thumb_metacarpals_base2, mass 0.00138588296544333; collision mesh filename=meshes/thumb_metacarpals_base2.STL; visual mesh filename=meshes/thumb_metacarpals_base2.STL
Joints:
- removed joint index_dip
- removed joint index_mcp_pitch
- removed joint middle_dip
- removed joint middle_mcp_pitch
- removed joint pinky_dip
- removed joint pinky_mcp_pitch
- removed joint ring_dip
- removed joint ring_mcp_pitch
- removed joint thumb_cmc_pitch
- removed joint thumb_cmc_yaw
- removed joint thumb_ip
- added joint lh_index_dip: type revolute, parent lh_index_proximal, child lh_index_distal, origin xyz=-0.0052516 0 0.036625 rpy=0 0 0, axis 0 1 0, limit lower=0 upper=1.43 effort=100 velocity=1, mimic joint=lh_index_mcp_pitch multiplier=0.89 offset=0
- added joint lh_index_mcp_pitch: type revolute, parent lh_hand_base_link, child lh_index_proximal, origin xyz=0.0024758 -0.02419 0.098779 rpy=0.05236 0 0, axis 0 1 0, limit lower=0 upper=1.60 effort=100 velocity=1
- added joint lh_middle_dip: type revolute, parent lh_middle_proximal, child lh_middle_distal, origin xyz=-0.0052516 0 0.036625 rpy=0 0 0, axis 0 1 0, limit lower=0 upper=1.43 effort=100 velocity=1, mimic joint=lh_middle_mcp_pitch multiplier=0.89 offset=0
- added joint lh_middle_mcp_pitch: type revolute, parent lh_hand_base_link, child lh_middle_proximal, origin xyz=0.00052576 -0.00634 0.1027 rpy=0 0 0, axis 0 1 0, limit lower=0 upper=1.60 effort=100 velocity=1
- added joint lh_pinky_dip: type revolute, parent lh_pinky_proximal, child lh_pinky_distal, origin xyz=-0.0052516 0 0.036625 rpy=0 0 0, axis 0 1 0, limit lower=0 upper=1.43 effort=100 velocity=1, mimic joint=lh_pinky_mcp_pitch multiplier=0.89 offset=0
- added joint lh_pinky_mcp_pitch: type revolute, parent lh_hand_base_link, child lh_pinky_proximal, origin xyz=0.0024758 0.028372 0.092741 rpy=-0.087266 0 0, axis 0 1 0, limit lower=0 upper=1.60 effort=100 velocity=1
- added joint lh_ring_dip: type revolute, parent lh_ring_proximal, child lh_ring_distal, origin xyz=-0.0052516 0 0.036625 rpy=0 0 0, axis 0 1 0, limit lower=0 upper=1.43 effort=100 velocity=1, mimic joint=lh_ring_mcp_pitch multiplier=0.89 offset=0
- added joint lh_ring_mcp_pitch: type revolute, parent lh_hand_base_link, child lh_ring_proximal, origin xyz=0.0010258 0.011135 0.098767 rpy=-0.05236 0 0, axis 0 1 0, limit lower=0 upper=1.60 effort=100 velocity=1
- added joint lh_thumb_cmc_pitch: type revolute, parent lh_thumb_metacarpals_base2, child lh_thumb_metacarpals, origin xyz=0.0061649 -0.010678 -0.004891 rpy=0 -1.1529 2.0944, axis 0 1 0, limit lower=0 upper=0.58 effort=100 velocity=1
- added joint lh_thumb_cmc_yaw: type revolute, parent lh_hand_base_link, child lh_thumb_metacarpals_base2, origin xyz=0.011508 -0.022975 0.032794 rpy=0 0 0, axis 0 0 1, limit lower=0 upper=1.3 effort=100 velocity=1
- added joint lh_thumb_ip: type revolute, parent lh_thumb_metacarpals, child lh_thumb_distal, origin xyz=0.0037776 0 0.045368 rpy=0 0 0, axis 0 1 0, limit lower=0 upper=1.08 effort=100 velocity=1, mimic joint=lh_thumb_cmc_pitch multiplier=2.29 offset=0

File: o6/right/linkerhand_o6_right.urdf (robot description, URDF)
Before this commit: robot linker_o6_right_v1.0_urdf, 12 links, 11 joints
Links:
- removed link hand_base_link
- removed link index_distal
- removed link index_proximal
- removed link middle_distal
- removed link middle_proximal
- removed link pinky_distal
- removed link pinky_proximal
- removed link ring_distal
- removed link ring_proximal
- removed link thumb_distal
- removed link thumb_metacarpals
- removed link thumb_metacarpals_base2
- added link rh_hand_base_link, mass 0.06740077960995; collision mesh filename=meshes/hand_base_link.STL; visual mesh filename=meshes/hand_base_link.STL
- added link rh_index_distal, mass 0.00376787129082313; collision mesh filename=meshes/index_distal.STL; visual mesh filename=meshes/index_distal.STL
- added link rh_index_proximal, mass 0.00253178529301663; collision mesh filename=meshes/index_proximal.STL; visual mesh filename=meshes/index_proximal.STL
- added link rh_middle_distal, mass 0.00376786259758948; collision mesh filename=meshes/middle_distal.STL; visual mesh filename=meshes/middle_distal.STL
- added link rh_middle_proximal, mass 0.00253175497594429; collision mesh filename=meshes/middle_proximal.STL; visual mesh filename=meshes/middle_proximal.STL
- added link rh_pinky_distal, mass 0.00376782669873412; collision mesh filename=meshes/pinky_distal.STL; visual mesh filename=meshes/pinky_distal.STL
- added link rh_pinky_proximal, mass 0.00253167400540778; collision mesh filename=meshes/pinky_proximal.STL; visual mesh filename=meshes/pinky_proximal.STL
- added link rh_ring_distal, mass 0.0037678395356105; collision mesh filename=meshes/ring_distal.STL; visual mesh filename=meshes/ring_distal.STL
- added link rh_ring_proximal, mass 0.00253170963529411; collision mesh filename=meshes/ring_proximal.STL; visual mesh filename=meshes/ring_proximal.STL
- added link rh_thumb_distal, mass 0.00763302603723749; collision mesh filename=meshes/thumb_distal.STL; visual mesh filename=meshes/thumb_distal.STL
- added link rh_thumb_metacarpals, mass 0.0123381607727595; collision mesh filename=meshes/thumb_metacarpals.STL; visual mesh filename=meshes/thumb_metacarpals.STL
- added link rh_thumb_metacarpals_base2, mass 0.00138591070212997; collision mesh filename=meshes/thumb_metacarpals_base2.STL; visual mesh filename=meshes/thumb_metacarpals_base2.STL
Joints:
- removed joint index_dip
- removed joint index_mcp_pitch
- removed joint middle_dip
- removed joint middle_mcp_pitch
- removed joint pinky_dip
- removed joint pinky_mcp_pitch
- removed joint ring_dip
- removed joint ring_mcp_pitch
- removed joint thumb_cmc_pitch
- removed joint thumb_cmc_yaw
- removed joint thumb_ip
- added joint rh_index_dip: type revolute, parent rh_index_proximal, child rh_index_distal, origin xyz=-0.0052516 0 0.036625 rpy=0 0 0, axis 0 1 0, limit lower=0 upper=1.43 effort=100 velocity=1, mimic joint=rh_index_mcp_pitch multiplier=0.89 offset=0
- added joint rh_index_mcp_pitch: type revolute, parent rh_hand_base_link, child rh_index_proximal, origin xyz=0.0024758 0.02419 0.098779 rpy=-0.05236 0 0, axis 0 1 0, limit lower=0 upper=1.60 effort=100 velocity=1
- added joint rh_middle_dip: type revolute, parent rh_middle_proximal, child rh_middle_distal, origin xyz=-0.0052516 0 0.036625 rpy=0 0 0, axis 0 1 0, limit lower=0 upper=1.43 effort=100 velocity=1, mimic joint=rh_middle_mcp_pitch multiplier=0.89 offset=0
- added joint rh_middle_mcp_pitch: type revolute, parent rh_hand_base_link, child rh_middle_proximal, origin xyz=0.00052576 0.00634 0.1027 rpy=0 0 0, axis 0 1 0, limit lower=0 upper=1.60 effort=100 velocity=1
- added joint rh_pinky_dip: type revolute, parent rh_pinky_proximal, child rh_pinky_distal, origin xyz=-0.0052516 0 0.036625 rpy=0 0 0, axis 0 1 0, limit lower=0 upper=1.43 effort=100 velocity=1, mimic joint=rh_pinky_mcp_pitch multiplier=0.89 offset=0
- added joint rh_pinky_mcp_pitch: type revolute, parent rh_hand_base_link, child rh_pinky_proximal, origin xyz=0.0024758 -0.028372 0.092741 rpy=0.087266 0 0, axis 0 1 0, limit lower=0 upper=1.60 effort=100 velocity=1
- added joint rh_ring_dip: type revolute, parent rh_ring_proximal, child rh_ring_distal, origin xyz=-0.0052516 0 0.036625 rpy=0 0 0, axis 0 1 0, limit lower=0 upper=1.43 effort=100 velocity=1, mimic joint=rh_ring_mcp_pitch multiplier=0.89 offset=0
- added joint rh_ring_mcp_pitch: type revolute, parent rh_hand_base_link, child rh_ring_proximal, origin xyz=0.0010258 -0.011135 0.098767 rpy=0.05236 0 0, axis 0 1 0, limit lower=0 upper=1.60 effort=100 velocity=1
- added joint rh_thumb_cmc_pitch: type revolute, parent rh_thumb_metacarpals_base2, child rh_thumb_metacarpals, origin xyz=0.0061649 0.010678 -0.004891 rpy=0 -1.1529 -2.0944, axis 0 1 0, limit lower=0 upper=0.58 effort=100 velocity=1
- added joint rh_thumb_cmc_yaw: type revolute, parent rh_hand_base_link, child rh_thumb_metacarpals_base2, origin xyz=0.011508 0.022975 0.032794 rpy=0 0 0, axis 0 0 -1, limit lower=0 upper=1.36 effort=100 velocity=1
- added joint rh_thumb_ip: type revolute, parent rh_thumb_metacarpals, child rh_thumb_distal, origin xyz=0.0037776 0 0.045368 rpy=0 0 0, axis 0 1 0, limit lower=0 upper=1.08 effort=100 velocity=1, mimic joint=rh_thumb_cmc_pitch multiplier=1.86 offset=0

Commit message: Updated left hand dynamics for all fingers. Updated kinematics for index_dip, middle_dip, ring_dip, and pinky_dip

File: l6/left/linkerhand_L6V3.1_left.urdf (robot description, URDF)
Before this commit: robot linkerhand_L6V3.1_left_2.1, 12 links, 11 joints
Joints:
- joint lh_index_dip: origin xyz=0.001001 -0.000537 0.028003 rpy=0 0 0 -> xyz=0.00093749 0 0.028002 rpy=0 0 0
- joint lh_middle_dip: origin xyz=0.000994 0.000058 0.028008 rpy=0 0 0 -> xyz=0.00093749 0 0.028002 rpy=0 0 0
- joint lh_pinky_dip: origin xyz=0.000979 0.001534 0.027967 rpy=0 0 0 -> xyz=0.00093749 0 0.028002 rpy=0 0 0
- joint lh_ring_dip: origin xyz=0.000979 0.001534 0.027967 rpy=0 0 0 -> xyz=0.00093749 0 0.028002 rpy=0 0 0
