Commit message: Added 'tip' coordinate origin for all fingers for L6

File: l6/left/linkerhand_L6V3.1_left.urdf (robot description, URDF)
Before this commit: robot linkerhand_L6V3.1_left_2.2, 12 links, 11 joints
Links:
- added link lh_index_tip
- added link lh_middle_tip
- added link lh_pinky_tip
- added link lh_ring_tip
- added link lh_thumb_tip
Joints:
- added joint lh_index_tip_fixed: type fixed, parent lh_index_distal, child lh_index_tip, origin xyz=0.0341 0 0.034 rpy=0 0 0
- added joint lh_middle_tip_fixed: type fixed, parent lh_middle_distal, child lh_middle_tip, origin xyz=0.0341 0 0.034 rpy=0 0 0
- added joint lh_pinky_tip_fixed: type fixed, parent lh_pinky_distal, child lh_pinky_tip, origin xyz=0.0341 0 0.034 rpy=0 0 0
- added joint lh_ring_tip_fixed: type fixed, parent lh_ring_distal, child lh_ring_tip, origin xyz=0.0341 0 0.034 rpy=0 0 0
- added joint lh_thumb_tip_fixed: type fixed, parent lh_thumb_distal, child lh_thumb_tip, origin xyz=0 0.0035 0.026 rpy=0 0 1.5708

File: l6/right/linkerhand_L6V3.1_right.urdf (robot description, URDF)
Before this commit: robot linkerhand_L6V3.1_right_2.2, 12 links, 11 joints
Links:
- added link rh_index_tip
- added link rh_middle_tip
- added link rh_pinky_tip
- added link rh_ring_tip
- added link rh_thumb_tip
Joints:
- added joint rh_index_tip_fixed: type fixed, parent rh_index_distal, child rh_index_tip, origin xyz=0.0341 0 0.034 rpy=0 0 0
- added joint rh_middle_tip_fixed: type fixed, parent rh_middle_distal, child rh_middle_tip, origin xyz=0.0341 0 0.034 rpy=0 0 0
- added joint rh_pinky_tip_fixed: type fixed, parent rh_pinky_distal, child rh_pinky_tip, origin xyz=0.0341 0 0.034 rpy=0 0 0
- added joint rh_ring_tip_fixed: type fixed, parent rh_ring_distal, child rh_ring_tip, origin xyz=0.0341 0 0.034 rpy=0 0 0
- added joint rh_thumb_tip_fixed: type fixed, parent rh_thumb_distal, child rh_thumb_tip, origin xyz=0 -0.0035 0.026 rpy=0 0 -1.5708

Commit message: Added mass and inertial parameters for fingertips as per PR comments

File: l6/left/linkerhand_L6V3.1_left.urdf (robot description, URDF)
Before this commit: robot linkerhand_L6V3.1_left_2.2, 17 links, 16 joints
Links:
- link lh_index_tip: mass None -> 1e-06
- link lh_middle_tip: mass None -> 1e-06
- link lh_pinky_tip: mass None -> 1e-06
- link lh_ring_tip: mass None -> 1e-06
- link lh_thumb_tip: mass None -> 1e-06

File: l6/right/linkerhand_L6V3.1_right.urdf (robot description, URDF)
Before this commit: robot linkerhand_L6V3.1_right_2.2, 17 links, 16 joints
Links:
- link rh_index_tip: mass None -> 1e-06
- link rh_middle_tip: mass None -> 1e-06
- link rh_pinky_tip: mass None -> 1e-06
- link rh_ring_tip: mass None -> 1e-06
- link rh_thumb_tip: mass None -> 1e-06
