Commit message: Updated L6 V3.1 URDF

File: l6/L6V3.1_left/linkerhand_L6V3.1_left.urdf (robot description, URDF)
Before this commit: robot linkerhand_L6V3.1_right, 12 links, 11 joints
Links:
- link hand_base_link: mass 0.989012019420379 -> 0.4185
- link index_distal: mass 0.989012019420379 -> 0.018408
- link index_proximal: mass 0.989012019420379 -> 0.008553
- link middle_distal: mass 0.989012019420379 -> 0.018408
- link middle_proximal: mass 0.989012019420379 -> 0.008553
- link pinky_distal: mass 0.989012019420379 -> 0.018408
- link pinky_proximal: mass 0.989012019420379 -> 0.008553
- link ring_distal: mass 0.989012019420379 -> 0.018408
- link ring_proximal: mass 0.989012019420379 -> 0.008553
- link thumb_distal: mass 0.989012019420379 -> 0.018
- link thumb_metacarpals: mass 0.989012019420379 -> 0.065
- link thumb_metacarpals_base1: mass 0.989012019420379 -> 0.01
Joints:
- removed joint thunb_cmc_roll
- added joint thumb_cmc_roll: type revolute, parent hand_base_link, child thumb_metacarpals_base1, origin xyz=0.0078133 -0.029898 0.026692 rpy=-0.034907 0 0, axis 0 0 1, limit lower=-0.087266 upper=1.256637 effort=0.588 velocity=5.95
- joint index_dip: limit lower=0 upper=1.14 effort=0 velocity=0 -> lower=0 upper=1.277039 effort=0 velocity=3.1; mimic joint=index_mcp_pitch multiplier=1.9 offset=0 -> joint=index_mcp_pitch multiplier=1.125676 offset=0; origin xyz=0.0012095 0 0.027992 rpy=0 0 0 -> xyz=0.001001 -0.000537 0.028003 rpy=0 0 0
- joint index_mcp_pitch: limit lower=0 upper=1.26 effort=0 velocity=0 -> lower=0 upper=1.134464 effort=0.574 velocity=6.10; origin xyz=-0.00066821 0.033041 0.11614 rpy=-0.087266 0 0 -> xyz=-0.00066821 -0.028967 0.11722 rpy=0 0 0
- joint middle_dip: limit lower=0 upper=1.14 effort=0 velocity=0 -> lower=0 upper=1.277039 effort=0 velocity=3.1; mimic joint=middle_mcp_pitch multiplier=1.9 offset=0 -> joint=middle_mcp_pitch multiplier=1.125676 offset=0; origin xyz=0.0009359 0 0.028002 rpy=0 0 0 -> xyz=0.000994 0.000058 0.028008 rpy=0 0 0
- joint middle_mcp_pitch: limit lower=0 upper=1.26 effort=0 velocity=0 -> lower=0 upper=1.134464 effort=0.574 velocity=6.10; origin xyz=-0.00066821 0.013196 0.12284 rpy=-0.034907 0 0 -> xyz=-0.00066821 -0.0089013 0.12322 rpy=0 0 0
- joint pinky_dip: limit lower=0 upper=1.14 effort=0 velocity=0 -> lower=0 upper=1.277039 effort=0 velocity=3.1; mimic joint=pinky_mcp_pitch multiplier=1.9 offset=0 -> joint=pinky_mcp_pitch multiplier=1.125676 offset=0; origin xyz=0.0009359 0 0.028002 rpy=0 0 0 -> xyz=0.000979 0.001534 0.027967 rpy=0 0 0
- joint pinky_mcp_pitch: limit lower=0 upper=1.26 effort=0 velocity=0 -> lower=0 upper=1.134464 effort=0.574 velocity=6.10; origin xyz=-0.00067852 -0.025809 0.11521 rpy=0.05236 0 -0.00010364 -> xyz=-0.00067852 0.029814 0.11424 rpy=0 0 0
- joint ring_dip: limit lower=0 upper=1.14 effort=0 velocity=0 -> lower=0 upper=1.277039 effort=0 velocity=3.1; mimic joint=ring_mcp_pitch multiplier=1.9 offset=0 -> joint=ring_mcp_pitch multiplier=1.125676 offset=0; origin xyz=0.0009359 0 0.028002 rpy=0 0 0 -> xyz=0.000979 0.001534 0.027967 rpy=0 0 0
- joint ring_mcp_pitch: limit lower=0 upper=1.26 effort=0 velocity=0 -> lower=0 upper=1.134464 effort=0.574 velocity=6.10; origin xyz=-0.00067368 -0.0065844 0.11852 rpy=0.017453 0 -0.00017259 -> xyz=-0.00067368 0.010717 0.11822 rpy=0 0 0
- joint thumb_cmc_pitch: axis 1 0 0 -> -1 0 0; limit lower=0 upper=0.99 effort=0 velocity=0 -> lower=0 upper=0.837758 effort=1.008 velocity=3.47; origin xyz=0.0081692 0.011981 0.00275 rpy=-1.4249 0 -0.61087 -> xyz=0.0057298 -0.01332 0.0027456 rpy=1.1083 0 0.40143
- joint thumb_dip: axis 1 0 0 -> -1 0 0; limit lower=0 upper=1.22 effort=0 velocity=0 -> lower=0 upper=0.963287 effort=0 velocity=1.7; mimic joint=thumb_cmc_pitch multiplier=2.22 offset=0 -> joint=thumb_cmc_pitch multiplier=1.226495 offset=0; origin xyz=0 -0.0061 0.0827 rpy=0 0 0 -> xyz=0 0.0061 0.0827 rpy=0 0 0
