Commit message: Update L25 URDF and meshes

File: l25/left/linkerhand_l25_left.urdf (robot description, URDF)
Before this commit: robot linkerhand_l25_left.urdf, 22 links, 21 joints
Links:
- link hand_base_link: mass 0.076924 -> 0.110373495507463
- link index_distal: mass 9.6249E-06 -> 0.00334170259772608
- link index_metacarpals: mass 0.0029534 -> 0.000895516429792169
- link index_middle: mass 4.0832E-06 -> 0.00237827499847615
- link index_proximal: mass 0.0093494 -> 0.00450921353606138
- link middle_distal: mass 9.6249E-06 -> 0.00334170288968694
- link middle_metacarpals: mass 0.0029534 -> 0.000895516947435045
- link middle_middle: mass 4.0832E-06 -> 0.00237827502274046
- link middle_proximal: mass 0.0093494 -> 0.00450921353536659
- link pinky_distal: mass 9.6249E-06 -> 0.00334170283969146
- link pinky_metacarpals: mass 0.0029534 -> 0.000895516947513541
- link pinky_middle: mass 4.0832E-06 -> 0.00237827431921004
- link pinky_proximal: mass 0.0093494 -> 0.00450921353949741
- link ring_distal: mass 9.6249E-06 -> 0.00334170280386792
- link ring_metacarpals: mass 0.0029534 -> 0.000895516612684195
- link ring_middle: mass 4.0832E-06 -> 0.00237827433282015
- link ring_proximal: mass 0.0093494 -> 0.00450921353946778
- link thumb_distal: mass 4.7117E-06 -> 0.00382046638843239
- link thumb_metacarpals: mass 0.019926 -> 0.0287160359417969
- link thumb_metacarpals_base1: mass 0.010336 -> 0.0160351802817401
- link thumb_metacarpals_base2: mass 0.002032 -> 0.00183264554882498
- link thumb_proximal: mass 0.0061013 -> 0.00549015507433734
Joints:
- joint index_dip: axis -1.5159E-05 1 0 -> 0 1 0; limit lower=0 upper=1.78 effort=0 velocity=0 -> lower=0 upper=1.55 effort=100 velocity=1; mimic (none) -> joint=index_pip multiplier=0.89 offset=0; origin xyz=0.00099206 -0.00025107 0.044322 rpy=0 0 0 -> xyz=0.0028245 0 0.031696 rpy=0 0 0
- joint index_mcp_pitch: axis 0 0.99998 -0.0056645 -> 0 1 0; limit lower=0 upper=1.68 effort=0 velocity=0 -> lower=0 upper=1.22 effort=100 velocity=1; origin xyz=0.0068598 -0.000102 0.018075 rpy=0 0 0 -> xyz=-0.0021302 0 0 rpy=0 0 0
- joint index_mcp_roll: limit lower=-0.24 upper=0.24 effort=0 velocity=0 -> lower=-0.23 upper=0.23 effort=100 velocity=1; origin xyz=0.0014994 -0.03367 0.13471 rpy=0 0 0 -> xyz=0.0038 -0.03525 0.1481 rpy=0 0 0
- joint index_pip: axis 0 0.99998 -0.0056645 -> 0 1 0; limit lower=0 upper=1.27 effort=0 velocity=0 -> lower=0 upper=1.74 effort=100 velocity=1; origin xyz=-0.0001598 -0.00024924 0.043999 rpy=0 0 0 -> xyz=-0.0041946 0 0.044819 rpy=0 0 0
- joint middle_dip: axis -1.5159E-05 1 0 -> 0 1 0; limit lower=0 upper=1.78 effort=0 velocity=0 -> lower=0 upper=1.55 effort=100 velocity=1; mimic (none) -> joint=middle_pip multiplier=0.89 offset=0; origin xyz=0.00099206 -0.00025107 0.044322 rpy=0 0 0 -> xyz=0.0028245 0 0.031696 rpy=0 0 0
- joint middle_mcp_pitch: axis 0 0.99998 -0.0056645 -> 0 1 0; limit lower=0 upper=1.68 effort=0 velocity=0 -> lower=0 upper=1.22 effort=100 velocity=1; origin xyz=0.0068598 -0.000102 0.018075 rpy=0 0 0 -> xyz=-0.0021302 0 0 rpy=0 0 0
- joint middle_mcp_roll: limit lower=-0.24 upper=0.24 effort=0 velocity=0 -> lower=-0.23 upper=0.23 effort=100 velocity=1; origin xyz=0.0014992 -0.01157 0.14219 rpy=0 0 0 -> xyz=0.00379999999265848 -0.0117500000029305 0.1526 rpy=0 0 0
- joint middle_pip: axis 0 0.99998 -0.0056645 -> 0 1 0; limit lower=0 upper=1.27 effort=0 velocity=0 -> lower=0 upper=1.74 effort=100 velocity=1; origin xyz=-0.0001598 -0.00024924 0.043999 rpy=0 0 0 -> xyz=-0.00419457745591796 0 0.0448194332262389 rpy=0 0 0
- joint pinky_dip: axis -1.5159E-05 1 0 -> 0 1 0; limit lower=0 upper=1.78 effort=0 velocity=0 -> lower=0 upper=1.55 effort=100 velocity=1; mimic (none) -> joint=pinky_pip multiplier=0.89 offset=0; origin xyz=0.00099206 -0.00025107 0.044322 rpy=0 0 0 -> xyz=0.0028245 0 0.031696 rpy=0 0 0
- joint pinky_mcp_pitch: axis 0 0.99998 -0.0056645 -> 0 1 0; limit lower=0 upper=1.68 effort=0 velocity=0 -> lower=0 upper=1.22 effort=100 velocity=1; origin xyz=0.0068598 -0.000102 0.018075 rpy=0 0 0 -> xyz=-0.0021302 0 0 rpy=0 0 0
- joint pinky_mcp_roll: limit lower=-0.24 upper=0.24 effort=0 velocity=0 -> lower=-0.23 upper=0.23 effort=100 velocity=1; origin xyz=0.0014989 0.03213 0.11977 rpy=0 0 0 -> xyz=0.00379999999998499 0.0352499999970695 0.1436 rpy=0 0 0
- joint pinky_pip: axis 0 0.99998 -0.0056645 -> 0 1 0; limit lower=0 upper=1.27 effort=0 velocity=0 -> lower=0 upper=1.74 effort=100 velocity=1; origin xyz=-0.0001598 -0.00024924 0.043999 rpy=0 0 0 -> xyz=-0.0041946 0 0.044819 rpy=0 0 0
- joint ring_dip: axis -1.5159E-05 1 0 -> 0 1 0; limit lower=0 upper=1.78 effort=0 velocity=0 -> lower=0 upper=1.55 effort=100 velocity=1; mimic (none) -> joint=ring_pip multiplier=0.89 offset=0; origin xyz=0.00099206 -0.00025107 0.044322 rpy=0 0 0 -> xyz=0.0028245 0 0.031696 rpy=0 0 0
- joint ring_mcp_pitch: axis 0 0.99998 -0.0056645 -> 0 1 0; limit lower=0 upper=1.68 effort=0 velocity=0 -> lower=0 upper=1.22 effort=100 velocity=1; origin xyz=0.0068598 -0.000102 0.018075 rpy=0 0 0 -> xyz=-0.0021302 0 0 rpy=0 0 0
- joint ring_mcp_roll: limit lower=-0.24 upper=0.24 effort=0 velocity=0 -> lower=-0.23 upper=0.23 effort=100 velocity=1; origin xyz=0.0014991 0.010029 0.13469 rpy=0 0 0 -> xyz=0.00379999999632174 0.0117499999970695 0.1481 rpy=0 0 0
- joint ring_pip: axis 0 0.99998 -0.0056645 -> 0 1 0; limit lower=0 upper=1.27 effort=0 velocity=0 -> lower=0 upper=1.74 effort=100 velocity=1; origin xyz=-0.0001598 -0.00024924 0.043999 rpy=0 0 0 -> xyz=-0.00419457745591796 0 0.0448194332262389 rpy=0 0 0
- joint thumb_cmc_pitch: axis -1 0 0 -> 0 1 0; limit lower=0 upper=1.59 effort=0 velocity=0 -> lower=0 upper=0.84 effort=100 velocity=1; origin xyz=0.006883 -0.014326 0.0014313 rpy=0 0 0 -> xyz=0.0088218 -0.024245 0.0005 rpy=0 -1.0647 1.9199
- joint thumb_cmc_roll: limit lower=-0.46 upper=0.61 effort=0 velocity=0 -> lower=0 upper=1.4 effort=100 velocity=1; origin xyz=-0.016601 -0.0024193 0.071265 rpy=0 0 0 -> xyz=0.01916 -0.01 0.0436 rpy=0 0 0
- joint thumb_cmc_yaw: axis 0 -0.0056645 0.99998 -> 0 0 1; limit lower=0 upper=1.57 effort=0 velocity=0 -> lower=0 upper=1.57 effort=100 velocity=1; origin xyz=0.04625 -0.0083829 -4.7486E-05 rpy=0 0 0 -> xyz=0.019845 0 0 rpy=0.77165 0 0
- joint thumb_ip: axis -1 0 0 -> 0 1 0; limit lower=0 upper=1.78 effort=0 velocity=0 -> lower=0 upper=1.29 effort=100 velocity=1; mimic (none) -> joint=thumb_mcp multiplier=1.02 offset=0; origin xyz=0 -0.046226 -0.0025751 rpy=0 0 0 -> xyz=-0.00483652209209624 0 0.0342226492098615 rpy=0 0 0
- joint thumb_mcp: axis -1 0 0 -> 0 1 0; limit lower=0 upper=1.59 effort=0 velocity=0 -> lower=0 upper=1.26 effort=100 velocity=1; origin xyz=0 -0.034219 -0.0041406 rpy=0 0 0 -> xyz=0.0127018248047608 0 0.0627256157349894 rpy=0 0 0

File: l25/right/linkerhand_l25_right.urdf (robot description, URDF)
Before this commit: robot linkerhand_l25_right.urdf, 22 links, 21 joints
Links:
- link hand_base_link: mass 0.077055 -> 0.130043890829375
- link index_distal: mass 9.6249E-06 -> 0.00334176238570705
- link index_metacarpals: mass 0.0029534 -> 0.000895533942236676
- link index_middle: mass 4.0832E-06 -> 0.00237861824163327
- link index_proximal: mass 0.0093494 -> 0.00450935628154297
- link middle_distal: mass 9.6249E-06 -> 0.0033417623857295
- link middle_metacarpals: mass 0.0029534 -> 0.000895533942236672
- link middle_middle: mass 4.0832E-06 -> 0.00237861824399121
- link middle_proximal: mass 0.0093494 -> 0.00450935628154299
- link pinky_distal: mass 9.6249E-06 -> 0.00334176233214274
- link pinky_metacarpals: mass 0.0029534 -> 0.000895533942236661
- link pinky_middle: mass 4.0832E-06 -> 0.0023786182416333
- link pinky_proximal: mass 0.0093494 -> 0.00450935627773312
- link ring_distal: mass 9.6249E-06 -> 0.00334176238553782
- link ring_metacarpals: mass 0.0029534 -> 0.00089553394223667
- link ring_middle: mass 4.0832E-06 -> 0.00237861824163314
- link ring_proximal: mass 0.0093494 -> 0.00450935628154299
- link thumb_distal: mass 4.7112E-06 -> 0.00585464206993151
- link thumb_metacarpals: mass 0.019929 -> 0.0311449727019751
- link thumb_metacarpals_base1: mass 0.010336 -> 0.0173128324517923
- link thumb_metacarpals_base2: mass 0.002032 -> 0.0129293097380942
- link thumb_proximal: mass 0.0061014 -> 0.00549015851204037
Joints:
- joint index_dip: limit lower=0 upper=1.78 effort=0 velocity=0 -> lower=0 upper=1.55 effort=1 velocity=100; mimic (none) -> joint=index_pip multiplier=0.89 offset=0; origin xyz=0.00099206 -0.00025106 0.044322 rpy=0 0 0 -> xyz=0.0028245 0 0.031696 rpy=0 0 0
- joint index_mcp_pitch: axis 0 0.99998 -0.0056645 -> 0 1 0; limit lower=0 upper=1.68 effort=0 velocity=0 -> lower=0 upper=1.22 effort=1 velocity=100; origin xyz=0.0068598 -0.00010189 0.018075 rpy=0 0 0 -> xyz=-0.0021302 0 0 rpy=0 0 0
- joint index_mcp_roll: limit lower=-0.24 upper=0.24 effort=0 velocity=0 -> lower=-0.23 upper=0.23 effort=1 velocity=100; origin xyz=0.0014984 0.032141 0.13508 rpy=0 0 0 -> xyz=0.0038 0.03525 0.1481 rpy=0 0 0
- joint index_pip: axis 0 0.99998 -0.0056645 -> 0 1 0; limit lower=0 upper=1.27 effort=0 velocity=0 -> lower=0 upper=1.75 effort=1 velocity=100; origin xyz=-0.0001598 -0.00024924 0.043999 rpy=0 0 0 -> xyz=-0.0041946 0 0.044819 rpy=0 0 0
- joint middle_dip: limit lower=0 upper=1.78 effort=0 velocity=0 -> lower=0 upper=1.55 effort=1 velocity=100; mimic (none) -> joint=middle_pip multiplier=0.89 offset=0; origin xyz=0.00099206 -0.00025106 0.044322 rpy=0 0 0 -> xyz=0.0028245 0 0.031696 rpy=0 0 0
- joint middle_mcp_pitch: axis 0 0.99998 -0.0056645 -> 0 1 0; limit lower=0 upper=1.68 effort=0 velocity=0 -> lower=0 upper=1.22 effort=1 velocity=100; origin xyz=0.0068598 -0.00010189 0.018075 rpy=0 0 0 -> xyz=-0.0021302 0 0 rpy=0 0 0
- joint middle_mcp_roll: limit lower=-0.24 upper=0.24 effort=0 velocity=0 -> lower=-0.23 upper=0.23 effort=1 velocity=100; origin xyz=0.0014985 0.0099581 0.14231 rpy=0 0 0 -> xyz=0.0038 0.01175 0.1526 rpy=0 0 0
- joint middle_pip: axis 0 0.99998 -0.0056645 -> 0 1 0; limit lower=0 upper=1.27 effort=0 velocity=0 -> lower=0 upper=1.75 effort=1 velocity=100; origin xyz=-0.0001598 -0.00024924 0.043999 rpy=0 0 0 -> xyz=-0.0041946 0 0.044819 rpy=0 0 0
- joint pinky_dip: limit lower=0 upper=1.78 effort=0 velocity=0 -> lower=0 upper=1.55 effort=1 velocity=100; mimic (none) -> joint=pinky_pip multiplier=0.89 offset=0; origin xyz=0.00099206 -0.00025106 0.044322 rpy=0 0 0 -> xyz=0.0028245 0 0.031696 rpy=0 0 0
- joint pinky_mcp_pitch: axis 0 0.99998 -0.0056645 -> 0 1 0; limit lower=0 upper=1.68 effort=0 velocity=0 -> lower=0 upper=1.22 effort=1 velocity=100; origin xyz=0.0068598 -0.00010189 0.018075 rpy=0 0 0 -> xyz=-0.0021302 0 0 rpy=0 0 0
- joint pinky_mcp_roll: limit lower=-0.24 upper=0.24 effort=0 velocity=0 -> lower=-0.23 upper=0.23 effort=1 velocity=100; origin xyz=0.0014989 -0.033485 0.1194 rpy=0 0 0 -> xyz=0.0038 -0.03525 0.1436 rpy=0 0 0
- joint pinky_pip: axis 0 0.99998 -0.0056645 -> 0 1 0; limit lower=0 upper=1.27 effort=0 velocity=0 -> lower=0 upper=1.75 effort=1 velocity=100; origin xyz=-0.0001598 -0.00024924 0.043999 rpy=0 0 0 -> xyz=-0.0041946 0 0.044819 rpy=0 0 0
- joint ring_dip: limit lower=0 upper=1.78 effort=0 velocity=0 -> lower=0 upper=1.55 effort=1 velocity=100; mimic (none) -> joint=ring_pip multiplier=0.89 offset=0; origin xyz=0.00099206 -0.00025106 0.044322 rpy=0 0 0 -> xyz=0.0028245 0 0.031696 rpy=0 0 0
- joint ring_mcp_pitch: axis 0 0.99998 -0.0056645 -> 0 1 0; limit lower=0 upper=1.68 effort=0 velocity=0 -> lower=0 upper=1.22 effort=1 velocity=100; origin xyz=0.0068598 -0.00010189 0.018075 rpy=0 0 0 -> xyz=-0.0021302 0 0 rpy=0 0 0
- joint ring_mcp_roll: limit lower=-0.24 upper=0.24 effort=0 velocity=0 -> lower=-0.23 upper=0.23 effort=1 velocity=100; origin xyz=0.0014987 -0.011555 0.13457 rpy=0 0 0 -> xyz=0.0038 -0.01175 0.1481 rpy=0 0 0
- joint ring_pip: axis 0 0.99998 -0.0056645 -> 0 1 0; limit lower=0 upper=1.27 effort=0 velocity=0 -> lower=0 upper=1.75 effort=1 velocity=100; origin xyz=-0.0001598 -0.00024924 0.043999 rpy=0 0 0 -> xyz=-0.0041946 0 0.044819 rpy=0 0 0
- joint thumb_cmc_pitch: axis 1 0 0 -> 0 1 0; limit lower=0 upper=1.59 effort=0 velocity=0 -> lower=0 upper=0.83 effort=1 velocity=100; origin xyz=0.006883 0.014309 0.0015936 rpy=0 0 0 -> xyz=0.0088264 0.024243 0.0005 rpy=0 -1.0647 -1.9199
- joint thumb_cmc_roll: limit lower=-0.46 upper=0.61 effort=0 velocity=0 -> lower=0 upper=1.39 effort=1 velocity=100; origin xyz=-0.016602 0.001612 0.071287 rpy=0 0 0 -> xyz=0.01916 0.01 0.0436 rpy=0 0 0
- joint thumb_cmc_yaw: axis 0 0.0056645 -0.99998 -> 0 0 -1; limit lower=0 upper=1.57 effort=0 velocity=0 -> lower=0 upper=1.57 effort=1 velocity=100; origin xyz=0.04625 0.0083829 4.7486E-05 rpy=0 0 0 -> xyz=0.019845 0 0 rpy=-0.77165 0 0
- joint thumb_ip: axis 1 0 0 -> 0 1 0; limit lower=0 upper=1.78 effort=0 velocity=0 -> lower=0 upper=1.29 effort=1 velocity=100; mimic (none) -> joint=thumb_mcp multiplier=1.03 offset=0; origin xyz=0 0.046252 -0.0020512 rpy=0 0 0 -> xyz=-0.0048365 0 0.034223 rpy=0 0 0
- joint thumb_mcp: axis 1 0 0 -> 0 1 0; limit lower=0- upper=1.59 effort=0 velocity=0 -> lower=0 upper=1.25 effort=1 velocity=100; origin xyz=0 0.034264 -0.0037526 rpy=0 0 0 -> xyz=0.012702 0 0.062726 rpy=0 0 0
