Commit message: chore: normalize lowercase paths and align urdf robot names

File: l25/left/linkerhand_l25_left.urdf (robot description, URDF)
Before this commit: robot linkerhand_o7v3_right, 18 links, 17 joints
Links:
- added link index_metacarpals, mass 0.000895516429792169; collision mesh filename=meshes/index_metacarpals.STL; visual mesh filename=meshes/index_metacarpals.STL
- added link middle_metacarpals, mass 0.000895516947435045; collision mesh filename=meshes/middle_metacarpals.STL; visual mesh filename=meshes/middle_metacarpals.STL
- added link pinky_metacarpals, mass 0.000895516947513541; collision mesh filename=meshes/pinky_metacarpals.STL; visual mesh filename=meshes/pinky_metacarpals.STL
- added link ring_metacarpals, mass 0.000895516612684195; collision mesh filename=meshes/ring_metacarpals.STL; visual mesh filename=meshes/ring_metacarpals.STL
- link hand_base_link: mass 0.115532510357281 -> 0.110373495507463
- link index_distal: mass 0.00314458616089874 -> 0.00334170259772608
- link index_middle: mass 0.00283043635989883 -> 0.00237827499847615
- link index_proximal: mass 0.00654982590538705 -> 0.00450921353606138
- link middle_distal: mass 0.00314458619941957 -> 0.00334170288968694
- link middle_middle: mass 0.00283043635989613 -> 0.00237827502274046
- link middle_proximal: mass 0.00654982976492332 -> 0.00450921353536659
- link pinky_distal: mass 0.00314458634356863 -> 0.00334170283969146
- link pinky_middle: mass 0.00283043635989883 -> 0.00237827431921004
- link pinky_proximal: mass 0.00654982590561137 -> 0.00450921353949741
- link ring_distal: mass 0.00314458625244518 -> 0.00334170280386792
- link ring_middle: mass 0.00283043635989883 -> 0.00237827433282015
- link ring_proximal: mass 0.00654982590560025 -> 0.00450921353946778
- link thumb_distal: mass 0.00512930046605133 -> 0.00382046638843239
- link thumb_metacarpals: mass 0.0152012310446388 -> 0.0287160359417969
- link thumb_metacarpals_base1: mass 0.0140456690808547 -> 0.0160351802817401
- link thumb_metacarpals_base2: mass 0.00582710539297639 -> 0.00183264554882498
- link thumb_proximal: mass 0.00662229628279784 -> 0.00549015507433734
Joints:
- added joint index_mcp_roll: type revolute, parent hand_base_link, child index_metacarpals, origin xyz=0.0038 -0.03525 0.1481 rpy=0 0 0, axis 1 0 0, limit lower=-0.23 upper=0.23 effort=100 velocity=1
- added joint middle_mcp_roll: type revolute, parent hand_base_link, child middle_metacarpals, origin xyz=0.00379999999265848 -0.0117500000029305 0.1526 rpy=0 0 0, axis 1 0 0, limit lower=-0.23 upper=0.23 effort=100 velocity=1
- added joint pinky_mcp_roll: type revolute, parent hand_base_link, child pinky_metacarpals, origin xyz=0.00379999999998499 0.0352499999970695 0.1436 rpy=0 0 0, axis 1 0 0, limit lower=-0.23 upper=0.23 effort=100 velocity=1
- added joint ring_mcp_roll: type revolute, parent hand_base_link, child ring_metacarpals, origin xyz=0.00379999999632174 0.0117499999970695 0.1481 rpy=0 0 0, axis 1 0 0, limit lower=-0.23 upper=0.23 effort=100 velocity=1
- joint index_dip: limit lower=0 upper=0.638 effort=100 velocity=1 -> lower=0 upper=1.55 effort=100 velocity=1; mimic joint=index_mcp_pitch multiplier=0.4615 offset=0 -> joint=index_pip multiplier=0.89 offset=0; origin xyz=-0.0052857 0 0.025703 rpy=0 0 0 -> xyz=0.0028245 0 0.031696 rpy=0 0 0
- joint index_mcp_pitch: limit lower=0 upper=1.3607 effort=100 velocity=1 -> lower=0 upper=1.22 effort=100 velocity=1; origin xyz=0.0022097 0.027177 0.12685 rpy=0 0 0 -> xyz=-0.0021302 0 0 rpy=0 0 0; parent hand_base_link -> index_metacarpals
- joint index_pip: limit lower=0 upper=1.8317 effort=100 velocity=1 -> lower=0 upper=1.74 effort=100 velocity=1; mimic joint=index_mcp_pitch multiplier=1.3462 offset=0 -> (none); origin xyz=-0.0010861 0 0.035634 rpy=0 0 0 -> xyz=-0.0041946 0 0.044819 rpy=0 0 0
- joint middle_dip: limit lower=0 upper=0.628 effort=100 velocity=1 -> lower=0 upper=1.55 effort=100 velocity=1; mimic joint=middle_mcp_pitch multiplier=0.4615 offset=0 -> joint=middle_pip multiplier=0.89 offset=0; origin xyz=-0.0052857 0 0.025703 rpy=0 0 0 -> xyz=0.0028245 0 0.031696 rpy=0 0 0
- joint middle_mcp_pitch: limit lower=0 upper=1.3607 effort=100 velocity=1 -> lower=0 upper=1.22 effort=100 velocity=1; origin xyz=0.0022097 0.0081771 0.13185 rpy=0 0 0 -> xyz=-0.0021302 0 0 rpy=0 0 0; parent hand_base_link -> middle_metacarpals
- joint middle_pip: limit lower=0 upper=1.8317 effort=100 velocity=1 -> lower=0 upper=1.74 effort=100 velocity=1; mimic joint=middle_mcp_pitch multiplier=1.3462 offset=0 -> (none); origin xyz=-0.0010861 0 0.035634 rpy=0 0 0 -> xyz=-0.00419457745591796 0 0.0448194332262389 rpy=0 0 0
- joint pinky_dip: limit lower=0 upper=0.628 effort=100 velocity=1 -> lower=0 upper=1.55 effort=100 velocity=1; mimic joint=pinky_mcp_pitch multiplier=0.4615 offset=0 -> joint=pinky_pip multiplier=0.89 offset=0; origin xyz=-0.0052857 0 0.025703 rpy=0 0 0 -> xyz=0.0028245 0 0.031696 rpy=0 0 0
- joint pinky_mcp_pitch: limit lower=0 upper=1.3607 effort=100 velocity=1 -> lower=0 upper=1.22 effort=100 velocity=1; origin xyz=0.0022097 -0.029823 0.12185 rpy=0 0 0 -> xyz=-0.0021302 0 0 rpy=0 0 0; parent hand_base_link -> pinky_metacarpals
- joint pinky_pip: limit lower=0 upper=1.8317 effort=100 velocity=1 -> lower=0 upper=1.74 effort=100 velocity=1; mimic joint=pinky_mcp_pitch multiplier=1.3462 offset=0 -> (none); origin xyz=-0.0010861 0 0.035634 rpy=0 0 0 -> xyz=-0.0041946 0 0.044819 rpy=0 0 0
- joint ring_dip: limit lower=0 upper=0.628 effort=100 velocity=1 -> lower=0 upper=1.55 effort=100 velocity=1; mimic joint=ring_mcp_pitch multiplier=0.4615 offset=0 -> joint=ring_pip multiplier=0.89 offset=0; origin xyz=-0.0052857 0 0.025703 rpy=0 0 0 -> xyz=0.0028245 0 0.031696 rpy=0 0 0
- joint ring_mcp_pitch: limit lower=0 upper=1.3607 effort=100 velocity=1 -> lower=0 upper=1.22 effort=100 velocity=1; origin xyz=0.0022097 -0.010823 0.12685 rpy=0 0 0 -> xyz=-0.0021302 0 0 rpy=0 0 0; parent hand_base_link -> ring_metacarpals
- joint ring_pip: limit lower=0 upper=1.8317 effort=100 velocity=1 -> lower=0 upper=1.74 effort=100 velocity=1; mimic joint=ring_mcp_pitch multiplier=1.3462 offset=0 -> (none); origin xyz=-0.0010861 0 0.035634 rpy=0 0 0 -> xyz=-0.00419457745591796 0 0.0448194332262389 rpy=0 0 0
- joint thumb_cmc_pitch: limit lower=0 upper=0.5146 effort=100 velocity=1 -> lower=0 upper=0.84 effort=100 velocity=1; origin xyz=0.00456 0.015168 -0.0019302 rpy=0 -0.9163 -1.8628 -> xyz=0.0088218 -0.024245 0.0005 rpy=0 -1.0647 1.9199
- joint thumb_cmc_roll: axis 1 0 0 -> -1 0 0; limit lower=0 upper=1.1339 effort=100 velocity=1 -> lower=0 upper=1.4 effort=100 velocity=1; origin xyz=-0.0116 0.018174 0.061651 rpy=0 0 0 -> xyz=0.01916 -0.01 0.0436 rpy=0 0 0
- joint thumb_cmc_yaw: axis 0 0 -1 -> 0 0 1; limit lower=0 upper=1.9189 effort=100 velocity=1 -> lower=0 upper=1.57 effort=100 velocity=1; origin xyz=0.0358 -0.00065771 0.0001518 rpy=-0.22683 0 0 -> xyz=0.019845 0 0 rpy=0.77165 0 0
- joint thumb_ip: limit lower=0 upper=0.7763 effort=100 velocity=1 -> lower=0 upper=1.29 effort=100 velocity=1; mimic joint=thumb_cmc_pitch multiplier=1.5085 offset=0 -> joint=thumb_mcp multiplier=1.02 offset=0; origin xyz=-0.00017064 0 0.038665 rpy=0 0 0 -> xyz=-0.00483652209209624 0 0.0342226492098615 rpy=0 0 0
- joint thumb_mcp: limit lower=0 upper=0.7152 effort=100 velocity=1 -> lower=0 upper=1.26 effort=100 velocity=1; mimic joint=thumb_cmc_pitch multiplier=1.3898 offset=0 -> (none); origin xyz=0.0061722 0 0.047968 rpy=0 0 0 -> xyz=0.0127018248047608 0 0.0627256157349894 rpy=0 0 0

File: l25/right/linkerhand_l25_right.urdf (robot description, URDF)
Before this commit: robot linkerhand_o7v3_right, 18 links, 17 joints
Links:
- added link index_metacarpals, mass 0.000895533942236676; collision mesh filename=meshes/index_metacarpals.STL; visual mesh filename=meshes/index_metacarpals.STL
- added link middle_metacarpals, mass 0.000895533942236672; collision mesh filename=meshes/middle_metacarpals.STL; visual mesh filename=meshes/middle_metacarpals.STL
- added link pinky_metacarpals, mass 0.000895533942236661; collision mesh filename=meshes/pinky_metacarpals.STL; visual mesh filename=meshes/pinky_metacarpals.STL
- added link ring_metacarpals, mass 0.00089553394223667; collision mesh filename=meshes/ring_metacarpals.STL; visual mesh filename=meshes/ring_metacarpals.STL
- link hand_base_link: mass 0.115532510357281 -> 0.130043890829375
- link index_distal: mass 0.00314458616089874 -> 0.00334176238570705
- link index_middle: mass 0.00283043635989883 -> 0.00237861824163327
- link index_proximal: mass 0.00654982590538705 -> 0.00450935628154297
- link middle_distal: mass 0.00314458619941957 -> 0.0033417623857295
- link middle_middle: mass 0.00283043635989613 -> 0.00237861824399121
- link middle_proximal: mass 0.00654982976492332 -> 0.00450935628154299
- link pinky_distal: mass 0.00314458634356863 -> 0.00334176233214274
- link pinky_middle: mass 0.00283043635989883 -> 0.0023786182416333
- link pinky_proximal: mass 0.00654982590561137 -> 0.00450935627773312
- link ring_distal: mass 0.00314458625244518 -> 0.00334176238553782
- link ring_middle: mass 0.00283043635989883 -> 0.00237861824163314
- link ring_proximal: mass 0.00654982590560025 -> 0.00450935628154299
- link thumb_distal: mass 0.00512930046605133 -> 0.00585464206993151
- link thumb_metacarpals: mass 0.0152012310446388 -> 0.0311449727019751
- link thumb_metacarpals_base1: mass 0.0140456690808547 -> 0.0173128324517923
- link thumb_metacarpals_base2: mass 0.00582710539297639 -> 0.0129293097380942
- link thumb_proximal: mass 0.00662229628279784 -> 0.00549015851204037
Joints:
- added joint index_mcp_roll: type revolute, parent hand_base_link, child index_metacarpals, origin xyz=0.0038 0.03525 0.1481 rpy=0 0 0, axis 1 0 0, limit lower=-0.23 upper=0.23 effort=1 velocity=100
- added joint middle_mcp_roll: type revolute, parent hand_base_link, child middle_metacarpals, origin xyz=0.0038 0.01175 0.1526 rpy=0 0 0, axis 1 0 0, limit lower=-0.23 upper=0.23 effort=1 velocity=100
- added joint pinky_mcp_roll: type revolute, parent hand_base_link, child pinky_metacarpals, origin xyz=0.0038 -0.03525 0.1436 rpy=0 0 0, axis 1 0 0, limit lower=-0.23 upper=0.23 effort=1 velocity=100
- added joint ring_mcp_roll: type revolute, parent hand_base_link, child ring_metacarpals, origin xyz=0.0038 -0.01175 0.1481 rpy=0 0 0, axis 1 0 0, limit lower=-0.23 upper=0.23 effort=1 velocity=100
- joint index_dip: limit lower=0 upper=0.638 effort=100 velocity=1 -> lower=0 upper=1.55 effort=1 velocity=100; mimic joint=index_mcp_pitch multiplier=0.4615 offset=0 -> joint=index_pip multiplier=0.89 offset=0; origin xyz=-0.0052857 0 0.025703 rpy=0 0 0 -> xyz=0.0028245 0 0.031696 rpy=0 0 0
- joint index_mcp_pitch: limit lower=0 upper=1.3607 effort=100 velocity=1 -> lower=0 upper=1.22 effort=1 velocity=100; origin xyz=0.0022097 0.027177 0.12685 rpy=0 0 0 -> xyz=-0.0021302 0 0 rpy=0 0 0; parent hand_base_link -> index_metacarpals
- joint index_pip: limit lower=0 upper=1.8317 effort=100 velocity=1 -> lower=0 upper=1.75 effort=1 velocity=100; mimic joint=index_mcp_pitch multiplier=1.3462 offset=0 -> (none); origin xyz=-0.0010861 0 0.035634 rpy=0 0 0 -> xyz=-0.0041946 0 0.044819 rpy=0 0 0
- joint middle_dip: limit lower=0 upper=0.628 effort=100 velocity=1 -> lower=0 upper=1.55 effort=1 velocity=100; mimic joint=middle_mcp_pitch multiplier=0.4615 offset=0 -> joint=middle_pip multiplier=0.89 offset=0; origin xyz=-0.0052857 0 0.025703 rpy=0 0 0 -> xyz=0.0028245 0 0.031696 rpy=0 0 0
- joint middle_mcp_pitch: limit lower=0 upper=1.3607 effort=100 velocity=1 -> lower=0 upper=1.22 effort=1 velocity=100; origin xyz=0.0022097 0.0081771 0.13185 rpy=0 0 0 -> xyz=-0.0021302 0 0 rpy=0 0 0; parent hand_base_link -> middle_metacarpals
- joint middle_pip: limit lower=0 upper=1.8317 effort=100 velocity=1 -> lower=0 upper=1.75 effort=1 velocity=100; mimic joint=middle_mcp_pitch multiplier=1.3462 offset=0 -> (none); origin xyz=-0.0010861 0 0.035634 rpy=0 0 0 -> xyz=-0.0041946 0 0.044819 rpy=0 0 0
- joint pinky_dip: limit lower=0 upper=0.628 effort=100 velocity=1 -> lower=0 upper=1.55 effort=1 velocity=100; mimic joint=pinky_mcp_pitch multiplier=0.4615 offset=0 -> joint=pinky_pip multiplier=0.89 offset=0; origin xyz=-0.0052857 0 0.025703 rpy=0 0 0 -> xyz=0.0028245 0 0.031696 rpy=0 0 0
- joint pinky_mcp_pitch: limit lower=0 upper=1.3607 effort=100 velocity=1 -> lower=0 upper=1.22 effort=1 velocity=100; origin xyz=0.0022097 -0.029823 0.12185 rpy=0 0 0 -> xyz=-0.0021302 0 0 rpy=0 0 0; parent hand_base_link -> pinky_metacarpals
- joint pinky_pip: limit lower=0 upper=1.8317 effort=100 velocity=1 -> lower=0 upper=1.75 effort=1 velocity=100; mimic joint=pinky_mcp_pitch multiplier=1.3462 offset=0 -> (none); origin xyz=-0.0010861 0 0.035634 rpy=0 0 0 -> xyz=-0.0041946 0 0.044819 rpy=0 0 0
- joint ring_dip: limit lower=0 upper=0.628 effort=100 velocity=1 -> lower=0 upper=1.55 effort=1 velocity=100; mimic joint=ring_mcp_pitch multiplier=0.4615 offset=0 -> joint=ring_pip multiplier=0.89 offset=0; origin xyz=-0.0052857 0 0.025703 rpy=0 0 0 -> xyz=0.0028245 0 0.031696 rpy=0 0 0
- joint ring_mcp_pitch: limit lower=0 upper=1.3607 effort=100 velocity=1 -> lower=0 upper=1.22 effort=1 velocity=100; origin xyz=0.0022097 -0.010823 0.12685 rpy=0 0 0 -> xyz=-0.0021302 0 0 rpy=0 0 0; parent hand_base_link -> ring_metacarpals
- joint ring_pip: limit lower=0 upper=1.8317 effort=100 velocity=1 -> lower=0 upper=1.75 effort=1 velocity=100; mimic joint=ring_mcp_pitch multiplier=1.3462 offset=0 -> (none); origin xyz=-0.0010861 0 0.035634 rpy=0 0 0 -> xyz=-0.0041946 0 0.044819 rpy=0 0 0
- joint thumb_cmc_pitch: limit lower=0 upper=0.5146 effort=100 velocity=1 -> lower=0 upper=0.83 effort=1 velocity=100; origin xyz=0.00456 0.015168 -0.0019302 rpy=0 -0.9163 -1.8628 -> xyz=0.0088264 0.024243 0.0005 rpy=0 -1.0647 -1.9199
- joint thumb_cmc_roll: limit lower=0 upper=1.1339 effort=100 velocity=1 -> lower=0 upper=1.39 effort=1 velocity=100; origin xyz=-0.0116 0.018174 0.061651 rpy=0 0 0 -> xyz=0.01916 0.01 0.0436 rpy=0 0 0
- joint thumb_cmc_yaw: limit lower=0 upper=1.9189 effort=100 velocity=1 -> lower=0 upper=1.57 effort=1 velocity=100; origin xyz=0.0358 -0.00065771 0.0001518 rpy=-0.22683 0 0 -> xyz=0.019845 0 0 rpy=-0.77165 0 0
- joint thumb_ip: limit lower=0 upper=0.7763 effort=100 velocity=1 -> lower=0 upper=1.29 effort=1 velocity=100; mimic joint=thumb_cmc_pitch multiplier=1.5085 offset=0 -> joint=thumb_mcp multiplier=1.03 offset=0; origin xyz=-0.00017064 0 0.038665 rpy=0 0 0 -> xyz=-0.0048365 0 0.034223 rpy=0 0 0
- joint thumb_mcp: limit lower=0 upper=0.7152 effort=100 velocity=1 -> lower=0 upper=1.25 effort=1 velocity=100; mimic joint=thumb_cmc_pitch multiplier=1.3898 offset=0 -> (none); origin xyz=0.0061722 0 0.047968 rpy=0 0 0 -> xyz=0.012702 0 0.062726 rpy=0 0 0
