Commit message: feat: Updated L20Lite URDF and meshes to match hardware release

File: l20lite/right/linkerhand_l20lite_right.urdf (robot description, URDF)
Before this commit: robot linkerhand_l20lite_right, 21 links, 20 joints
Links:
- link hand_base_link: mass 0.10884427610512 -> 0.108844276105116
- link index_distal: mass 0.00314458657125681 -> 0.0031446130611452
- link index_metacarpals: mass 0.00903700347459462 -> 0.00903700329493157
- link index_middle: mass 0.00283043635595588 -> 0.00283043630937165
- link index_proximal: mass 0.00654982479821771 -> 0.00654982235507964
- link middle_distal: mass 0.0031445865911477 -> 0.00314458659113992
- link middle_middle: mass 0.00283043635504843 -> 0.00283043635504842
- link middle_proximal: mass 0.00654982478226948 -> 0.00654982478226949
- link pinky_distal: mass 0.0031445864920905 -> 0.00314457409502053
- link pinky_metacarpals: mass 0.00903700347459465 -> 0.00903700307878998
- link pinky_middle: mass 0.00283043635595589 -> 0.00283043670305552
- link pinky_proximal: mass 0.00654982918810593 -> 0.00654983474179372
- link ring_distal: mass 0.0031445863941225 -> 0.00314460631735109
- link ring_metacarpals: mass 0.00903700347459463 -> 0.00903700335356623
- link ring_middle: mass 0.00283043628669241 -> 0.0028304363455826
- link ring_proximal: mass 0.00654982867950541 -> 0.00654983629670871
- link thumb_distal: mass 0.00512933613321634 -> 0.00512919991432349
- link thumb_metacarpals: mass 0.0152011697874328 -> 0.0152012256765109
- link thumb_metacarpals_base1: mass 0.0084581719416891 -> 0.0084581547726202
- link thumb_metacarpals_base2: mass 0.00582710536801184 -> 0.00582711245702963
- link thumb_proximal: mass 0.00662230120907192 -> 0.00662231923284161
Joints:
- joint index_dip: limit lower=0 upper=1.8317 effort=100 velocity=1 -> lower=0 upper=0.62 effort=10.43 velocity=1; mimic joint=index_mcp_pitch multiplier=0.4616 offset=0 -> joint=index_mcp_pitch multiplier=0.46 offset=0; origin xyz=-0.0054686 0 0.025665 rpy=0 0 0 -> xyz=-0.0052444 0 0.025711 rpy=0 0 0
- joint index_mcp_pitch: limit lower=0 upper=1.3607 effort=100 velocity=1 -> lower=0 upper=1.36 effort=4.8 velocity=1; origin xyz=0.0020763 0 0.015294 rpy=0 0 0 -> xyz=0.00220968332188026 0 0.0152749792820048 rpy=0 0 0
- joint index_mcp_roll: axis -0.99996 0 0.0087265 -> -1 0 0; limit lower=0 upper=0.2181 effort=100 velocity=1 -> lower=0 upper=0.19 effort=100 velocity=1; origin xyz=-0.0021643 0.026654 0.13253 rpy=0 0 0 -> xyz=-0.0021643 0.026654 0.13253 rpy=-0.027925 -0.0087266 0
- joint index_pip: limit lower=0 upper=1.8317 effort=100 velocity=1 -> lower=0 upper=1.78 effort=3.7 velocity=1; mimic joint=index_mcp_pitch multiplier=1.3462 offset=0 -> joint=index_mcp_pitch multiplier=1.3 offset=0; origin xyz=-0.0013807 0 0.035624 rpy=0 0 0 -> xyz=-0.0010697 0 0.035634 rpy=0 0 0
- joint middle_dip: limit lower=0 upper=0.628 effort=100 velocity=1 -> lower=0 upper=0.62 effort=10.43 velocity=1; mimic joint=middle_mcp_pitch multiplier=0.4616 offset=0 -> joint=middle_mcp_pitch multiplier=0.46 offset=0
- joint middle_mcp_pitch: limit lower=0 upper=1.3607 effort=100 velocity=1 -> lower=0 upper=1.36 effort=100 velocity=1; origin xyz=-0.0021316 0.0076542 0.15281 rpy=0 0 0 -> xyz=-0.00213155528434806 0.00765417737818821 0.152810108410232 rpy=0 0 0
- joint middle_pip: limit lower=0 upper=1.8317 effort=100 velocity=1 -> lower=0 upper=1.78 effort=3.7 velocity=1; mimic joint=middle_mcp_pitch multiplier=1.3462 offset=0 -> joint=middle_mcp_pitch multiplier=1.3 offset=0; origin xyz=-0.001397 0 0.035623 rpy=0 0 0 -> xyz=-0.00139702428111229 0 0.0356230829860553 rpy=0 0 0
- joint pinky_dip: limit lower=0 upper=0.628 effort=100 velocity=1 -> lower=0 upper=0.62 effort=10.43 velocity=1; mimic joint=pinky_mcp_pitch multiplier=0.4616 offset=0 -> joint=pinky_mcp_pitch multiplier=0.46 offset=0; origin xyz=-0.0054686 0 0.025665 rpy=0 0 0 -> xyz=-0.0052444 0 0.025711 rpy=0 0 0
- joint pinky_mcp_pitch: limit lower=0 upper=1.3607 effort=100 velocity=1 -> lower=0 upper=1.36 effort=4.8 velocity=1; origin xyz=0.0020763 0 0.015294 rpy=0 0 0 -> xyz=0.0022097 0 0.015275 rpy=0 0 0
- joint pinky_mcp_roll: axis 0.99996 0 0.0087265 -> 1 0 0; limit lower=0 upper=0.3489 effort=100 velocity=1 -> lower=0 upper=0.3 effort=4.29 velocity=1; origin xyz=-0.00012074 -0.030346 0.12755 rpy=0 0 0 -> xyz=-0.00012074 -0.030346 0.12755 rpy=0.057596 -0.0087266 0
- joint pinky_pip: limit lower=0 upper=1.8317 effort=100 velocity=1 -> lower=0 upper=1.78 effort=3.7 velocity=1; mimic joint=pinky_mcp_pitch multiplier=1.3462 offset=0 -> joint=pinky_mcp_pitch multiplier=1.34 offset=0; origin xyz=-0.0013807 0 0.035624 rpy=0 0 0 -> xyz=-0.0010697 0 0.035634 rpy=0 0 0
- joint ring_dip: axis 0 1 0 -> 0.000213099161087669 0.999450193223668 -0.033155178387707; limit lower=0 upper=0.628 effort=100 velocity=1 -> lower=0 upper=0.62 effort=10.43 velocity=1; mimic joint=ring_mcp_pitch multiplier=0.4616 offset=0 -> joint=ring_mcp_pitch multiplier=0.46 offset=0; origin xyz=-0.0054686 0 0.025665 rpy=0 0 0 -> xyz=-0.00524443259686075 0 0.0257114125710868 rpy=0 0 -0.000213216385347256
- joint ring_mcp_pitch: limit lower=0 upper=1.3607 effort=100 velocity=1 -> lower=0 upper=1.36 effort=4.8 velocity=1; origin xyz=0.0020763 0 0.015294 rpy=0 0 0 -> xyz=0.0022097 0 0.015275 rpy=0 0 0
- joint ring_mcp_roll: axis 0.99996 0 0.0087265 -> 1 0 0; limit lower=0 upper=0.2181 effort=100 velocity=1 -> lower=0 upper=0.2 effort=4.29 velocity=1; origin xyz=-0.0021643 -0.011346 0.13253 rpy=0 0 0 -> xyz=-0.00216430029569533 -0.0113458226218121 0.132534071328313 rpy=0.0244346095279086 -0.00872664625996829 0
- joint ring_pip: limit lower=0 upper=1.8317 effort=100 velocity=1 -> lower=0 upper=1.78 effort=3.7 velocity=1; mimic joint=ring_mcp_pitch multiplier=1.3462 offset=0 -> joint=ring_mcp_pitch multiplier=1.34 offset=0; origin xyz=-0.0013807 0 0.035624 rpy=0 0 0 -> xyz=-0.00106974956301328 0 0.0356344124989653 rpy=0 0 0
- joint thumb_cmc_pitch: limit lower=0 upper=0.5146 effort=100 velocity=1 -> lower=0 upper=0.52 effort=4.8 velocity=1; origin xyz=0.0046051 0.014383 -0.0051478 rpy=0.16356 -1.1191 -2.0038 -> xyz=0.0037151 0.015396 -0.0019302 rpy=0 -0.9163 -1.8076
- joint thumb_cmc_roll: limit lower=0 upper=1.1339 effort=100 velocity=1 -> lower=0 upper=1.03 effort=4.8 velocity=1
- joint thumb_cmc_yaw: axis 0.008517 -0.21782 -0.97595 -> 0 0 -1; limit lower=0 upper=1.9189 effort=100 velocity=0 -> lower=0 upper=1.40 effort=4.8 velocity=1; origin xyz=0.035797 -0.00065879 0.00045944 rpy=0 0 0 -> xyz=0.035798 -0.0006691 0.00040146 rpy=-0.13233 -0.0085747 0.0011413
- joint thumb_ip: limit lower=0 upper=0.7763 effort=100 velocity=1 -> lower=0 upper=0.78 effort=3.36 velocity=1; mimic joint=thumb_cmc_pitch multiplier=1.508 offset=0 -> joint=thumb_cmc_pitch multiplier=1.49 offset=0
- joint thumb_mcp: limit lower=0 upper=0.7152 effort=100 velocity=1 -> lower=0 upper=0.72 effort=3.7 velocity=1; mimic joint=thumb_cmc_pitch multiplier=1.3898 offset=0 -> joint=thumb_cmc_pitch multiplier=1.38 offset=0
