Commit message: Update O6 URDF and meshes to 1014_v4
Import both URDFs and referenced GLB visual/OBJ collision payloads from linker-bot/linker-sim-assets at e6bcf44ff0203534e14500cb836f57e9f9492292. Replace superseded STL assets and adopt mirrored geometry, corrected thumb frames, and hardware inertial parameters.

File: O6/left/linkerhand_o6_left.urdf (robot description, URDF)
Before this commit: robot linkerhand_o6_left, 12 links, 11 joints
Links:
- link lh_hand_base_link: mass 0.0672935238166485 -> 0.2374; geometry collision mesh filename=meshes/collision/lh_hand_base_link_col.obj; visual mesh filename=meshes/visual/lh_hand_base_link_vis.glb
- link lh_index_distal: mass 0.00376951085886838 -> 0.00632; geometry collision mesh filename=meshes/collision/lh_index_distal_col.obj; visual mesh filename=meshes/visual/lh_index_distal_vis.glb
- link lh_index_proximal: mass 0.00253174651934627 -> 0.01082; geometry collision mesh filename=meshes/collision/lh_index_proximal_col.obj; visual mesh filename=meshes/visual/lh_index_proximal_vis.glb
- link lh_middle_distal: mass 0.00376952789210256 -> 0.00632; geometry collision mesh filename=meshes/collision/lh_middle_distal_col.obj; visual mesh filename=meshes/visual/lh_middle_distal_vis.glb
- link lh_middle_proximal: mass 0.00253177375206983 -> 0.01082; geometry collision mesh filename=meshes/collision/lh_middle_proximal_col.obj; visual mesh filename=meshes/visual/lh_middle_proximal_vis.glb
- link lh_pinky_distal: mass 0.00376948071276134 -> 0.00632; geometry collision mesh filename=meshes/collision/lh_pinky_distal_col.obj; visual mesh filename=meshes/visual/lh_pinky_distal_vis.glb
- link lh_pinky_proximal: mass 0.00253185993162408 -> 0.01082; geometry collision mesh filename=meshes/collision/lh_pinky_proximal_col.obj; visual mesh filename=meshes/visual/lh_pinky_proximal_vis.glb
- link lh_ring_distal: mass 0.00376949588316609 -> 0.00632; geometry collision mesh filename=meshes/collision/lh_ring_distal_col.obj; visual mesh filename=meshes/visual/lh_ring_distal_vis.glb
- link lh_ring_proximal: mass 0.00253182223645066 -> 0.01082; geometry collision mesh filename=meshes/collision/lh_ring_proximal_col.obj; visual mesh filename=meshes/visual/lh_ring_proximal_vis.glb
- link lh_thumb_distal: mass 0.00763332957284057 -> 0.0142; geometry collision mesh filename=meshes/collision/lh_thumb_distal_col.obj; visual mesh filename=meshes/visual/lh_thumb_distal_vis.glb
- link lh_thumb_metacarpals: mass 0.0123381586619931 -> 0.04724; geometry collision mesh filename=meshes/collision/lh_thumb_metacarpals_col.obj; visual mesh filename=meshes/visual/lh_thumb_metacarpals_vis.glb
- link lh_thumb_metacarpals_base2: mass 0.00138588296544333 -> 0.00258; geometry collision mesh filename=meshes/collision/lh_thumb_metacarpals_base2_col.obj; visual mesh filename=meshes/visual/lh_thumb_metacarpals_base2_vis.glb
Joints:
- joint lh_index_dip: axis 0 1 0 -> 0.0 1.0 0.0; limit lower=0 upper=1.43 effort=100 velocity=1 -> lower=0.0 upper=1.43 effort=100 velocity=1; mimic joint=lh_index_mcp_pitch multiplier=0.89 offset=0 -> joint=lh_index_mcp_pitch multiplier=0.89 offset=0.0; origin xyz=-0.0052516 0 0.036625 rpy=0 0 0 -> xyz=-0.0052516 -0.0 0.036625 rpy=-0.0 -0.0 -0.0
- joint lh_index_mcp_pitch: axis 0 1 0 -> 0.0 1.0 0.0; limit lower=0 upper=1.60 effort=100 velocity=1 -> lower=0.0 upper=1.6 effort=100 velocity=1; origin xyz=0.0024758 -0.02419 0.098779 rpy=0.05236 0 0 -> xyz=0.0024758 -0.02419 0.098779 rpy=0.05236 -0.0 -0.0
- joint lh_middle_dip: axis 0 1 0 -> 0.0 1.0 0.0; limit lower=0 upper=1.43 effort=100 velocity=1 -> lower=0.0 upper=1.43 effort=100 velocity=1; mimic joint=lh_middle_mcp_pitch multiplier=0.89 offset=0 -> joint=lh_middle_mcp_pitch multiplier=0.89 offset=0.0; origin xyz=-0.0052516 0 0.036625 rpy=0 0 0 -> xyz=-0.0052516 -0.0 0.036625 rpy=-0.0 -0.0 -0.0
- joint lh_middle_mcp_pitch: axis 0 1 0 -> 0.0 1.0 0.0; limit lower=0 upper=1.60 effort=100 velocity=1 -> lower=0.0 upper=1.6 effort=100 velocity=1; origin xyz=0.00052576 -0.00634 0.1027 rpy=0 0 0 -> xyz=0.00052576 -0.00634 0.1027 rpy=-0.0 -0.0 -0.0
- joint lh_pinky_dip: axis 0 1 0 -> 0.0 1.0 0.0; limit lower=0 upper=1.43 effort=100 velocity=1 -> lower=0.0 upper=1.43 effort=100 velocity=1; mimic joint=lh_pinky_mcp_pitch multiplier=0.89 offset=0 -> joint=lh_pinky_mcp_pitch multiplier=0.89 offset=0.0; origin xyz=-0.0052516 0 0.036625 rpy=0 0 0 -> xyz=-0.0052516 -0.0 0.036625 rpy=-0.0 -0.0 -0.0
- joint lh_pinky_mcp_pitch: axis 0 1 0 -> 0.0 1.0 0.0; limit lower=0 upper=1.60 effort=100 velocity=1 -> lower=0.0 upper=1.6 effort=100 velocity=1; origin xyz=0.0024758 0.028372 0.092741 rpy=-0.087266 0 0 -> xyz=0.0024758 0.028372 0.092741 rpy=-0.087266 -0.0 -0.0
- joint lh_ring_dip: axis 0 1 0 -> 0.0 1.0 0.0; limit lower=0 upper=1.43 effort=100 velocity=1 -> lower=0.0 upper=1.43 effort=100 velocity=1; mimic joint=lh_ring_mcp_pitch multiplier=0.89 offset=0 -> joint=lh_ring_mcp_pitch multiplier=0.89 offset=0.0; origin xyz=-0.0052516 0 0.036625 rpy=0 0 0 -> xyz=-0.0052516 -0.0 0.036625 rpy=-0.0 -0.0 -0.0
- joint lh_ring_mcp_pitch: axis 0 1 0 -> 0.0 1.0 0.0; limit lower=0 upper=1.60 effort=100 velocity=1 -> lower=0.0 upper=1.6 effort=100 velocity=1; origin xyz=0.0010258 0.011135 0.098767 rpy=-0.05236 0 0 -> xyz=0.0010258 0.011135 0.098767 rpy=-0.05236 -0.0 -0.0
- joint lh_thumb_cmc_pitch: axis 0 1 0 -> -1.0 -0.0 -0.0; limit lower=0 upper=0.58 effort=100 velocity=1 -> lower=0.0 upper=0.58 effort=100 velocity=1; origin xyz=0.0061649 -0.010678 -0.004891 rpy=0 -1.1529 2.0944 -> xyz=0.0061649 -0.010678 -0.004891 rpy=1.1529 -0.0 0.5236
- joint lh_thumb_cmc_yaw: axis 0 0 1 -> -0.0 -0.0 1.0; limit lower=0 upper=1.3 effort=100 velocity=1 -> lower=0.0 upper=1.36 effort=100 velocity=1; origin xyz=0.011508 -0.022975 0.032794 rpy=0 0 0 -> xyz=0.010457 -0.022975 0.030794 rpy=-0.0 -0.0 -0.0
- joint lh_thumb_ip: axis 0 1 0 -> -1.0 -0.0 -0.0; limit lower=0 upper=1.08 effort=100 velocity=1 -> lower=0.0 upper=1.08 effort=100 velocity=1; mimic joint=lh_thumb_cmc_pitch multiplier=2.29 offset=0 -> joint=lh_thumb_cmc_pitch multiplier=1.86 offset=0.0; origin xyz=0.0037776 0 0.045368 rpy=0 0 0 -> xyz=0.0 0.0037776 0.045368 rpy=-0.0 -0.0 -0.0

File: O6/right/linkerhand_o6_right.urdf (robot description, URDF)
Before this commit: robot linkerhand_o6_right, 12 links, 11 joints
Links:
- link rh_hand_base_link: mass 0.06740077960995 -> 0.2374; geometry collision mesh filename=meshes/collision/rh_hand_base_link_col.obj; visual mesh filename=meshes/visual/rh_hand_base_link_vis.glb
- link rh_index_distal: mass 0.00376787129082313 -> 0.00632; geometry collision mesh filename=meshes/collision/rh_index_distal_col.obj; visual mesh filename=meshes/visual/rh_index_distal_vis.glb
- link rh_index_proximal: mass 0.00253178529301663 -> 0.01082; geometry collision mesh filename=meshes/collision/rh_index_proximal_col.obj; visual mesh filename=meshes/visual/rh_index_proximal_vis.glb
- link rh_middle_distal: mass 0.00376786259758948 -> 0.00632; geometry collision mesh filename=meshes/collision/rh_middle_distal_col.obj; visual mesh filename=meshes/visual/rh_middle_distal_vis.glb
- link rh_middle_proximal: mass 0.00253175497594429 -> 0.01082; geometry collision mesh filename=meshes/collision/rh_middle_proximal_col.obj; visual mesh filename=meshes/visual/rh_middle_proximal_vis.glb
- link rh_pinky_distal: mass 0.00376782669873412 -> 0.00632; geometry collision mesh filename=meshes/collision/rh_pinky_distal_col.obj; visual mesh filename=meshes/visual/rh_pinky_distal_vis.glb
- link rh_pinky_proximal: mass 0.00253167400540778 -> 0.01082; geometry collision mesh filename=meshes/collision/rh_pinky_proximal_col.obj; visual mesh filename=meshes/visual/rh_pinky_proximal_vis.glb
- link rh_ring_distal: mass 0.0037678395356105 -> 0.00632; geometry collision mesh filename=meshes/collision/rh_ring_distal_col.obj; visual mesh filename=meshes/visual/rh_ring_distal_vis.glb
- link rh_ring_proximal: mass 0.00253170963529411 -> 0.01082; geometry collision mesh filename=meshes/collision/rh_ring_proximal_col.obj; visual mesh filename=meshes/visual/rh_ring_proximal_vis.glb
- link rh_thumb_distal: mass 0.00763302603723749 -> 0.0142; geometry collision mesh filename=meshes/collision/rh_thumb_distal_col.obj; visual mesh filename=meshes/visual/rh_thumb_distal_vis.glb
- link rh_thumb_metacarpals: mass 0.0123381607727595 -> 0.04724; geometry collision mesh filename=meshes/collision/rh_thumb_metacarpals_col.obj; visual mesh filename=meshes/visual/rh_thumb_metacarpals_vis.glb
- link rh_thumb_metacarpals_base2: mass 0.00138591070212997 -> 0.00258; geometry collision mesh filename=meshes/collision/rh_thumb_metacarpals_base2_col.obj; visual mesh filename=meshes/visual/rh_thumb_metacarpals_base2_vis.glb
Joints:
- joint rh_thumb_cmc_pitch: axis 0 1 0 -> 1 0 0; origin xyz=0.0061649 0.010678 -0.004891 rpy=0 -1.1529 -2.0944 -> xyz=0.0061649 0.010678 -0.004891 rpy=-1.1529 0 -0.5236
- joint rh_thumb_cmc_yaw: origin xyz=0.011508 0.022975 0.032794 rpy=0 0 0 -> xyz=0.010457 0.022975 0.030794 rpy=0 0 0
- joint rh_thumb_ip: axis 0 1 0 -> 1 0 0; origin xyz=0.0037776 0 0.045368 rpy=0 0 0 -> xyz=0 -0.0037776 0.045368 rpy=0 0 0
